File: cad/gpi-ctl.sch (EAGLE design)
At the start: 91 parts, among them CN2 MICROSDPLAIN, CN3 1X4-BIG, IC1 7803SR, SW1 SWITCHGT12-THOLE, SW2 SWITCHKMR211, SW3 SWITCHKMR211, U1 STM32F4/64, U2 ACS711, U3 ULN2003, U8 IC_FT230X-SSOP-16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

Commit message: regulator
Parts:
- removed IC1: 7803SR, adafruit:7805T
- added C36: (no value), jaw:C0603
- added C37: 10u, jaw:C0603
- added J4: 1X4-BIG, adafruit:1X4-BIG
- added VREG1: ROF-78E3.3-0.5, jaw:REGULATORROF
- added VREG2: MCP1824, jaw:MCP1824
Connections:
- new net N$8: D2.C, VREG2.NSHTDN, VREG2.VIN
- net GND: now also C36.P$2, C37.P$2, J4.2, VREG1.GND, VREG2.GND; no longer IC1.GND
- net I2CC: now also J4.4
- net I2CD: now also J4.3
- net VCC: now also C36.P$1, C37.P$1, J4.1, VREG1.VO, VREG2.VOUT; no longer IC1.VO
- net VCCM: now also VREG1.VI; no longer IC1.VI
- net VIN: no longer D2.C
Changed lines of the file:
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@@
 <part name="D1" library="jaw" deviceset="DIODE" device="SOD-323"/>
 <part name="VCC14" library="jaw" deviceset="PWR-VCC" device=""/>
-<part name="IC1" library="adafruit" deviceset="78*" device="T" technology="05" value="7803SR"/>
+<part name="VREG1" library="jaw" deviceset="REGULATOR" device="ROF" value=" ROF-78E3.3-0.5"/>
 <part name="C1" library="jaw" deviceset="C" device="0603" value="10u"/>
 <part name="C2" library="jaw" deviceset="C" device="1210" value="100u"/>
@@
 <part name="C35" library="jaw" deviceset="C" device="0603" value=".1u"/>
 <part name="U$1" library="jaw" deviceset="ROBOTMAN-LOGO" device=""/>
+<part name="VREG2" library="jaw" deviceset="MCP1824" device=""/>
+<part name="GND20" library="jaw" deviceset="PWR-GND" device=""/>
+<part name="VCC12" library="jaw" deviceset="PWR-VCC" device=""/>
+<part name="C36" library="jaw" deviceset="C" device="0603"/>
+<part name="C37" library="jaw" deviceset="C" device="0603" value="10u"/>
+<part name="J4" library="adafruit" deviceset="1X4" device="-BIG"/>
+<part name="VCC13" library="jaw" deviceset="PWR-VCC" device=""/>
+<part name="GND21" library="jaw" deviceset="PWR-GND" device=""/>
 </parts>
 <sheets>
@@
 <instance part="D1" gate="G$1" x="327.66" y="248.92" rot="R90"/>
 <instance part="VCC14" gate="G$1" x="337.82" y="264.16"/>
-<instance part="IC1" gate="A1" x="66.04" y="55.88"/>
+<instance part="VREG1" gate="G$1" x="66.04" y="55.88"/>
 <instance part="C1" gate="G$1" x="48.26" y="50.8"/>
 <instance part="C2" gate="G$1" x="83.82" y="50.8"/>
@@
 <instance part="C35" gate="G$1" x="27.94" y="251.46"/>
 <instance part="U$1" gate="G$1" x="314.96" y="7.62"/>
+<instance part="VREG2" gate="G$1" x="350.52" y="73.66"/>
+<instance part="GND20" gate="G$1" x="350.52" y="60.96"/>
+<instance part="VCC12" gate="G$1" x="373.38" y="78.74"/>
+<instance part="C36" gate="G$1" x="373.38" y="71.12"/>
+<instance part="C37" gate="G$1" x="22.86" y="251.46"/>
+<instance part="J4" gate="G$1" x="355.6" y="182.88"/>
+<instance part="VCC13" gate="G$1" x="332.74" y="190.5"/>
+<instance part="GND21" gate="G$1" x="332.74" y="175.26"/>
 </instances>
 <busses>
@@
 </segment>
 <segment>
-<pinref part="IC1" gate="A1" pin="GND"/>
+<pinref part="VREG1" gate="G$1" pin="GND"/>
 <pinref part="GND2" gate="G$1" pin="GND"/>
-<wire x1="66.04" y1="48.26" x2="66.04" y2="45.72" width="0.1524" layer="91"/>
 <pinref part="C1" gate="G$1" pin="P$2"/>
 <wire x1="66.04" y1="45.72" x2="66.04" y2="40.64" width="0.1524" layer="91"/>
@@
 <junction x="33.02" y="248.92"/>
 <junction x="38.1" y="248.92"/>
+<pinref part="C37" gate="G$1" pin="P$2"/>
+<wire x1="22.86" y1="248.92" x2="27.94" y2="248.92" width="0.1524" layer="91"/>
+<junction x="27.94" y="248.92"/>
 </segment>
 <segment>
@@
 <wire x1="355.6" y1="157.48" x2="350.52" y2="157.48" width="0.1524" layer="91"/>
 <junction x="350.52" y="157.48"/>
+</segment>
+<segment>
+<pinref part="VREG2" gate="G$1" pin="GND"/>
+<pinref part="GND20" gate="G$1" pin="GND"/>
+<wire x1="350.52" y1="63.5" x2="350.52" y2="66.04" width="0.1524" layer="91"/>
+<pinref part="C36" gate="G$1" pin="P$2"/>
+<wire x1="373.38" y1="68.58" x2="373.38" y2="66.04" width="0.1524" layer="91"/>
+<wire x1="373.38" y1="66.04" x2="350.52" y2="66.04" width="0.1524" layer="91"/>
+<junction x="350.52" y="66.04"/>
+</segment>
+<segment>
+<pinref part="GND21" gate="G$1" pin="GND"/>
+<pinref part="J4" gate="G$1" pin="2"/>
+<wire x1="332.74" y1="177.8" x2="332.74" y2="182.88" width="0.1524" layer="91"/>
+<wire x1="332.74" y1="182.88" x2="350.52" y2="182.88" width="0.1524" layer="91"/>
 </segment>
 </net>
@@
 <segment>
 <pinref part="C2" gate="G$1" pin="P$1"/>
-<pinref part="IC1" gate="A1" pin="VO"/>
-<wire x1="83.82" y1="55.88" x2="76.2" y2="55.88" width="0.1524" layer="91"/>
+<pinref part="VREG1" gate="G$1" pin="VO"/>
+<wire x1="83.82" y1="55.88" x2="78.74" y2="55.88" width="0.1524" layer="91"/>
 <pinref part="C3" gate="G$1" pin="P$1"/>
 <wire x1="83.82" y1="55.88" x2="88.9" y2="55.88" width="0.1524" layer="91"/>
@@
 <junction x="33.02" y="256.54"/>
 <junction x="38.1" y="256.54"/>
+<pinref part="C37" gate="G$1" pin="P$1"/>
+<wire x1="22.86" y1="256.54" x2="27.94" y2="256.54" width="0.1524" layer="91"/>
+<junction x="27.94" y="256.54"/>
 </segment>
 <segment>
@@
 <wire x1="363.22" y1="154.94" x2="388.62" y2="154.94" width="0.1524" layer="91"/>
 <wire x1="388.62" y1="154.94" x2="388.62" y2="157.48" width="0.1524" layer="91"/>
+</segment>
+<segment>
+<pinref part="VCC12" gate="G$1" pin="VCC"/>
+<pinref part="C36" gate="G$1" pin="P$1"/>
+<pinref part="VREG2" gate="G$1" pin="VOUT"/>
+<wire x1="365.76" y1="76.2" x2="373.38" y2="76.2" width="0.1524" layer="91"/>
+<junction x="373.38" y="76.2"/>
+</segment>
+<segment>
+<pinref part="VCC13" gate="G$1" pin="VCC"/>
+<pinref part="J4" gate="G$1" pin="1"/>
+<wire x1="332.74" y1="187.96" x2="332.74" y2="185.42" width="0.1524" layer="91"/>
+<wire x1="332.74" y1="185.42" x2="350.52" y2="185.42" width="0.1524" layer="91"/>
 </segment>
 </net>
@@
 <net name="VCCM" class="0">
 <segment>
-<pinref part="IC1" gate="A1" pin="VI"/>
+<pinref part="VREG1" gate="G$1" pin="VI"/>
 <pinref part="C1" gate="G$1" pin="P$1"/>
-<wire x1="48.26" y1="55.88" x2="55.88" y2="55.88" width="0.1524" layer="91"/>
+<wire x1="48.26" y1="55.88" x2="53.34" y2="55.88" width="0.1524" layer="91"/>
 <junction x="48.26" y="55.88"/>
 <pinref part="VCCM1" gate="G$1" pin="VCCM"/>
@@
 <pinref part="CN3" gate="G$1" pin="3"/>
 </segment>
-<segment>
-<pinref part="D2" gate="G$1" pin="C"/>
-<wire x1="304.8" y1="76.2" x2="314.96" y2="76.2" width="0.1524" layer="91"/>
-<label x="312.42" y="76.2" size="1.778" layer="95"/>
-</segment>
 </net>
 <net name="ADC2" class="0">
@@
 <label x="264.16" y="172.72" size="1.778" layer="95"/>
 </segment>
+<segment>
+<pinref part="J4" gate="G$1" pin="4"/>
+<wire x1="350.52" y1="177.8" x2="345.44" y2="177.8" width="0.1524" layer="91"/>
+</segment>
 </net>
 <net name="I2CD" class="0">
@@
 <wire x1="259.08" y1="170.18" x2="264.16" y2="170.18" width="0.1524" layer="91"/>
 <label x="264.16" y="170.18" size="1.778" layer="95"/>
+</segment>
+<segment>
+<pinref part="J4" gate="G$1" pin="3"/>
+<wire x1="350.52" y1="180.34" x2="345.44" y2="180.34" width="0.1524" layer="91"/>
 </segment>
 </net>
@@
 </segment>
 </net>
+<net name="N$8" class="0">
+<segment>
+<pinref part="VREG2" gate="G$1" pin="VIN"/>
+<pinref part="D2" gate="G$1" pin="C"/>
+<wire x1="335.28" y1="76.2" x2="332.74" y2="76.2" width="0.1524" layer="91"/>
+<pinref part="VREG2" gate="G$1" pin="NSHTDN"/>
+<wire x1="332.74" y1="76.2" x2="304.8" y2="76.2" width="0.1524" layer="91"/>
+<wire x1="335.28" y1="73.66" x2="332.74" y2="73.66" width="0.1524" layer="91"/>
+<wire x1="332.74" y1="73.66" x2="332.74" y2="76.2" width="0.1524" layer="91"/>
+<junction x="332.74" y="76.2"/>
+</segment>
+</net>

Commit message: tweak sent to fab
Parts:
- C36: value (none) -> 10u
Changed lines of the file:
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@@
 <setting verticaltext="up"/>
 </settings>
-<grid distance="0.1" unitdist="inch" unit="inch" style="lines" multiple="1" display="yes" altdistance="0.01" altunitdist="inch" altunit="inch"/>
+<grid distance="0.1" unitdist="inch" unit="inch" style="lines" multiple="1" display="no" altdistance="0.01" altunitdist="inch" altunit="inch"/>
 <layers>
 <layer number="1" name="Top" color="4" fill="1" visible="no" active="no"/>
@@
 <part name="GND20" library="jaw" deviceset="PWR-GND" device=""/>
 <part name="VCC12" library="jaw" deviceset="PWR-VCC" device=""/>
-<part name="C36" library="jaw" deviceset="C" device="0603"/>
+<part name="C36" library="jaw" deviceset="C" device="0603" value="10u"/>
 <part name="C37" library="jaw" deviceset="C" device="0603" value="10u"/>
 <part name="J4" library="adafruit" deviceset="1X4" device="-BIG"/>

Commit message: tweak text
Parts:
- C1: value 10u -> 10u 25V
- LED1: value (none) -> green
- LED2: value (none) -> red
- LED3: value (none) -> white
Changed lines of the file:
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@@
 <setting verticaltext="up"/>
 </settings>
-<grid distance="0.1" unitdist="inch" unit="inch" style="lines" multiple="1" display="yes" altdistance="0.01" altunitdist="inch" altunit="inch"/>
+<grid distance="0.1" unitdist="inch" unit="inch" style="lines" multiple="1" display="no" altdistance="0.01" altunitdist="inch" altunit="inch"/>
 <layers>
 <layer number="1" name="Top" color="4" fill="1" visible="no" active="no"/>
@@
 <part name="VCC14" library="jaw" deviceset="PWR-VCC" device=""/>
 <part name="VREG1" library="jaw" deviceset="REGULATOR" device="ROF" value=" ROF-78E3.3-0.5"/>
-<part name="C1" library="jaw" deviceset="C" device="0603" value="10u"/>
+<part name="C1" library="jaw" deviceset="C" device="0603" value="10u 25V"/>
 <part name="C2" library="jaw" deviceset="C" device="1210" value="100u"/>
 <part name="C3" library="jaw" deviceset="C" device="0603" value="1u"/>
@@
 <part name="VCC5" library="jaw" deviceset="PWR-VCC" device=""/>
 <part name="SW1" library="jaw" deviceset="SWITCH" device="GT12-THOLE"/>
-<part name="LED1" library="adafruit" deviceset="LED" device="3MM"/>
-<part name="LED2" library="adafruit" deviceset="LED" device="3MM"/>
-<part name="LED3" library="adafruit" deviceset="LED" device="3MM"/>
+<part name="LED1" library="adafruit" deviceset="LED" device="3MM" value="green"/>
+<part name="LED2" library="adafruit" deviceset="LED" device="3MM" value="red"/>
+<part name="LED3" library="adafruit" deviceset="LED" device="3MM" value="white"/>
 <part name="C25" library="jaw" deviceset="C" device="0603" value=".1u"/>
 <part name="VCC6" library="jaw" deviceset="PWR-VCC" device=""/>

Commit message: temp sensor
Parts:
- added C38: (no value), jaw:C0603
- added R15: (no value), jaw:R0603
Connections:
- new net N$9: R15.P$1, U4.OUT
- net ADCTMP: now also C38.P$1, R15.P$2; no longer U4.OUT
- net GND: now also C38.P$2
Changed lines of the file:
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@@
 <?xml version="1.0" encoding="utf-8"?>
 <!DOCTYPE eagle SYSTEM "eagle.dtd">
-<eagle version="7.0.1">
+<eagle version="7.1.0">
 <drawing>
 <settings>
@@
 <setting verticaltext="up"/>
 </settings>
-<grid distance="0.1" unitdist="inch" unit="inch" style="lines" multiple="1" display="no" altdistance="0.01" altunitdist="inch" altunit="inch"/>
+<grid distance="0.1" unitdist="inch" unit="inch" style="lines" multiple="1" display="yes" altdistance="0.01" altunitdist="inch" altunit="inch"/>
 <layers>
 <layer number="1" name="Top" color="4" fill="1" visible="no" active="no"/>
@@
 <part name="VCC13" library="jaw" deviceset="PWR-VCC" device=""/>
 <part name="GND21" library="jaw" deviceset="PWR-GND" device=""/>
+<part name="R15" library="jaw" deviceset="R" device="0603"/>
+<part name="C38" library="jaw" deviceset="C" device="0603"/>
 </parts>
 <sheets>
@@
 <instance part="VCC13" gate="G$1" x="332.74" y="190.5"/>
 <instance part="GND21" gate="G$1" x="332.74" y="175.26"/>
+<instance part="R15" gate="G$1" x="93.98" y="251.46"/>
+<instance part="C38" gate="G$1" x="101.6" y="246.38"/>
 </instances>
 <busses>
@@
 <wire x1="71.12" y1="243.84" x2="81.28" y2="243.84" width="0.1524" layer="91"/>
 <junction x="81.28" y="243.84"/>
+<pinref part="C38" gate="G$1" pin="P$2"/>
+<wire x1="101.6" y1="243.84" x2="81.28" y2="243.84" width="0.1524" layer="91"/>
 </segment>
 <segment>
@@
 </segment>
 <segment>
-<pinref part="U4" gate="G$1" pin="OUT"/>
-<wire x1="88.9" y1="251.46" x2="93.98" y2="251.46" width="0.1524" layer="91"/>
-<label x="91.44" y="251.46" size="1.778" layer="95"/>
+<pinref part="R15" gate="G$1" pin="P$2"/>
+<pinref part="C38" gate="G$1" pin="P$1"/>
+<wire x1="99.06" y1="251.46" x2="101.6" y2="251.46" width="0.1524" layer="91"/>
+<wire x1="101.6" y1="251.46" x2="109.22" y2="251.46" width="0.1524" layer="91"/>
+<junction x="101.6" y="251.46"/>
+<label x="106.68" y="251.46" size="1.778" layer="95"/>
 </segment>
 </net>
@@
 </segment>
 </net>
+<net name="N$9" class="0">
+<segment>
+<pinref part="U4" gate="G$1" pin="OUT"/>
+<pinref part="R15" gate="G$1" pin="P$1"/>
+</segment>
+</net>
