File: cad/gpi-ctl.sch (EAGLE design)
At the start: 99 parts, among them CN2 MICROSDPLAIN, CN3 1X4-BIG, J4 1X4-BIG, SW1 SWITCHGT12-THOLE, SW2 SWITCHKMR211, SW3 SWITCHKMR211, U1 STM32F4/64, U2 ACS711, U3 ULN2003, U5 max4452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

Commit message: vcca to conn
Parts:
- added C33: 1u, jaw:C0603
- C11, C12: value .001u -> .1u
- C13, C14: value .001u -> 1u
- C38: value (none) -> 1u
- C40: value 1u -> .1u
- R15: value (none) -> 100
Connections:
- net GND: now also C33.P$2
- net VCC: no longer C31.P$1, J1.P$6, U4.V
- net VCCA: now also C31.P$1, C33.P$1, J1.P$6, U4.V
Other:
- note added: "II"
- note added: "IO"
- note added: "Tb"
- note added: "Tt"
- note added: "VH"
- note added: "VO"
Changed lines of the file:
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@@
 <part name="D8" library="jaw" deviceset="ZENER" device="" value="4v"/>
 <part name="C10" library="jaw" deviceset="C" device="0603" value=".001u"/>
-<part name="C11" library="jaw" deviceset="C" device="0603" value=".001u"/>
-<part name="C12" library="jaw" deviceset="C" device="0603" value=".001u"/>
-<part name="C13" library="jaw" deviceset="C" device="0603" value=".001u"/>
-<part name="C14" library="jaw" deviceset="C" device="0603" value=".001u"/>
+<part name="C11" library="jaw" deviceset="C" device="0603" value=".1u"/>
+<part name="C12" library="jaw" deviceset="C" device="0603" value=".1u"/>
+<part name="C13" library="jaw" deviceset="C" device="0603" value="1u"/>
+<part name="C14" library="jaw" deviceset="C" device="0603" value="1u"/>
 <part name="C17" library="jaw" deviceset="C" device="0603" value=".001u"/>
 <part name="R1" library="jaw" deviceset="R" device="0603" value="100"/>
@@
 <part name="GND5" library="jaw" deviceset="PWR-GND" device=""/>
 <part name="VCCM7" library="jaw" deviceset="PWR-VCCM" device=""/>
-<part name="VCC3" library="jaw" deviceset="PWR-VCC" device=""/>
 <part name="J1" library="jaw" deviceset="HEADER-2X4" device=""/>
 <part name="J2" library="jaw" deviceset="HEADER-2X4" device=""/>
@@
 <part name="U3" library="jaw" deviceset="ULN2003" device=""/>
 <part name="U4" library="jaw" deviceset="TEMPERATURE" device=""/>
-<part name="VCC8" library="jaw" deviceset="PWR-VCC" device=""/>
 <part name="GND19" library="jaw" deviceset="PWR-GND" device=""/>
 <part name="C31" library="jaw" deviceset="C" device="0603" value=".1u"/>
@@
 <part name="VCC13" library="jaw" deviceset="PWR-VCC" device=""/>
 <part name="GND21" library="jaw" deviceset="PWR-GND" device=""/>
-<part name="R15" library="jaw" deviceset="R" device="0603"/>
-<part name="C38" library="jaw" deviceset="C" device="0603"/>
+<part name="R15" library="jaw" deviceset="R" device="0603" value="100"/>
+<part name="C38" library="jaw" deviceset="C" device="0603" value="1u"/>
 <part name="U5" library="jaw" deviceset="OPAMP" device="" value="max4452"/>
 <part name="R19" library="jaw" deviceset="R" device="0603" value="22"/>
@@
 <part name="VCC16" library="jaw" deviceset="PWR-VCC" device=""/>
 <part name="R20" library="jaw" deviceset="R" device="0603" value="100"/>
-<part name="C40" library="jaw" deviceset="C" device="0603" value="1u"/>
+<part name="C40" library="jaw" deviceset="C" device="0603" value=".1u"/>
+<part name="C33" library="jaw" deviceset="C" device="0603" value="1u"/>
+<part name="GND28" library="jaw" deviceset="PWR-GND" device=""/>
+<part name="VCCA3" library="jaw" deviceset="PWR-VCCA" device=""/>
+<part name="VCCA5" library="jaw" deviceset="PWR-VCCA" device=""/>
+<part name="VCCA6" library="jaw" deviceset="PWR-VCCA" device=""/>
 </parts>
 <sheets>
@@
 <text x="182.88" y="114.3" size="3.81" layer="97">M471-OLED display</text>
 <text x="271.78" y="124.46" size="3.81" layer="97">SD CARD</text>
+<text x="35.56" y="198.12" size="2.54" layer="97">II</text>
+<text x="53.34" y="198.12" size="2.54" layer="97">VH</text>
+<text x="71.12" y="198.12" size="2.54" layer="97">VO</text>
+<text x="88.9" y="198.12" size="2.54" layer="97">Tb</text>
+<text x="106.68" y="198.12" size="2.54" layer="97">Tt</text>
+<text x="124.46" y="198.12" size="2.54" layer="97">IO</text>
 </plain>
 <instances>
@@
 <instance part="GND5" gate="G$1" x="332.74" y="157.48"/>
 <instance part="VCCM7" gate="G$1" x="381" y="162.56"/>
-<instance part="VCC3" gate="G$1" x="388.62" y="160.02"/>
 <instance part="J1" gate="A" x="358.14" y="154.94"/>
 <instance part="J2" gate="A" x="358.14" y="139.7"/>
@@
 <instance part="U3" gate="G$1" x="317.5" y="215.9"/>
 <instance part="U4" gate="G$1" x="81.28" y="251.46"/>
-<instance part="VCC8" gate="G$1" x="81.28" y="264.16"/>
 <instance part="GND19" gate="G$1" x="81.28" y="238.76"/>
 <instance part="C31" gate="G$1" x="71.12" y="251.46"/>
@@
 <instance part="R20" gate="G$1" x="139.7" y="25.4"/>
 <instance part="C40" gate="G$1" x="147.32" y="17.78"/>
+<instance part="C33" gate="G$1" x="25.4" y="223.52"/>
+<instance part="GND28" gate="G$1" x="25.4" y="218.44"/>
+<instance part="VCCA3" gate="G$1" x="25.4" y="231.14"/>
+<instance part="VCCA5" gate="G$1" x="388.62" y="160.02"/>
+<instance part="VCCA6" gate="G$1" x="81.28" y="264.16"/>
 </instances>
 <busses>
@@
 <wire x1="91.44" y1="15.24" x2="111.76" y2="15.24" width="0.1524" layer="91"/>
 </segment>
+<segment>
+<pinref part="C33" gate="G$1" pin="P$2"/>
+<pinref part="GND28" gate="G$1" pin="GND"/>
+</segment>
 </net>
 <net name="VCC" class="0">
@@
 </segment>
 <segment>
-<pinref part="U4" gate="G$1" pin="V"/>
-<pinref part="VCC8" gate="G$1" pin="VCC"/>
-<wire x1="81.28" y1="261.62" x2="81.28" y2="259.08" width="0.1524" layer="91"/>
-<pinref part="C31" gate="G$1" pin="P$1"/>
-<wire x1="71.12" y1="256.54" x2="71.12" y2="259.08" width="0.1524" layer="91"/>
-<wire x1="71.12" y1="259.08" x2="81.28" y2="259.08" width="0.1524" layer="91"/>
-<junction x="81.28" y="259.08"/>
-</segment>
-<segment>
 <pinref part="FAN1" gate="J" pin="3"/>
 <wire x1="363.22" y1="241.3" x2="360.68" y2="241.3" width="0.1524" layer="91"/>
@@
 </segment>
 <segment>
-<pinref part="J1" gate="A" pin="P$6"/>
-<pinref part="VCC3" gate="G$1" pin="VCC"/>
-<wire x1="363.22" y1="154.94" x2="388.62" y2="154.94" width="0.1524" layer="91"/>
-<wire x1="388.62" y1="154.94" x2="388.62" y2="157.48" width="0.1524" layer="91"/>
-</segment>
-<segment>
 <pinref part="VCC12" gate="G$1" pin="VCC"/>
 <pinref part="C36" gate="G$1" pin="P$1"/>
@@
 <junction x="124.46" y="55.88"/>
 </segment>
+<segment>
+<pinref part="C33" gate="G$1" pin="P$1"/>
+<pinref part="VCCA3" gate="G$1" pin="VCCA"/>
+</segment>
+<segment>
+<pinref part="J1" gate="A" pin="P$6"/>
+<wire x1="363.22" y1="154.94" x2="388.62" y2="154.94" width="0.1524" layer="91"/>
+<wire x1="388.62" y1="154.94" x2="388.62" y2="157.48" width="0.1524" layer="91"/>
+<pinref part="VCCA5" gate="G$1" pin="VCCA"/>
+</segment>
+<segment>
+<pinref part="U4" gate="G$1" pin="V"/>
+<wire x1="81.28" y1="261.62" x2="81.28" y2="259.08" width="0.1524" layer="91"/>
+<pinref part="C31" gate="G$1" pin="P$1"/>
+<wire x1="71.12" y1="256.54" x2="71.12" y2="259.08" width="0.1524" layer="91"/>
+<wire x1="71.12" y1="259.08" x2="81.28" y2="259.08" width="0.1524" layer="91"/>
+<junction x="81.28" y="259.08"/>
+<pinref part="VCCA6" gate="G$1" pin="VCCA"/>
+</segment>
 </net>

Commit message: sync, green led
Parts:
- added CN1: HEADER-1X2.4, jaw:HEADER-1X2.4
- R9: value 1k -> 470
Connections:
- new net N$12: CN1.P$2, U1.PA6
- net GND: now also CN1.P$1
- net IOLED1: now also U1.PC9; no longer U1.PA6
Other:
- note added: "Sync Out"
Changed lines of the file:
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@@
 <part name="J2" library="jaw" deviceset="HEADER-2X4" device=""/>
 <part name="J3" library="jaw" deviceset="HEADER-2X4" device=""/>
-<part name="R9" library="jaw" deviceset="R" device="0603" value="1k"/>
+<part name="R9" library="jaw" deviceset="R" device="0603" value="470"/>
 <part name="R11" library="jaw" deviceset="R" device="0603" value="1k"/>
 <part name="R12" library="jaw" deviceset="R" device="0603" value="1k"/>
@@
 <part name="VCCA5" library="jaw" deviceset="PWR-VCCA" device=""/>
 <part name="VCCA6" library="jaw" deviceset="PWR-VCCA" device=""/>
+<part name="CN1" library="jaw" deviceset="HEADER-1X2" device=".4" value="HEADER-1X2.4"/>
+<part name="GND29" library="jaw" deviceset="PWR-GND" device=""/>
 </parts>
 <sheets>
@@
 <text x="106.68" y="198.12" size="2.54" layer="97">Tt</text>
 <text x="124.46" y="198.12" size="2.54" layer="97">IO</text>
+<text x="165.1" y="170.18" size="2.54" layer="97">Sync Out</text>
 </plain>
 <instances>
@@
 <instance part="VCCA5" gate="G$1" x="388.62" y="160.02"/>
 <instance part="VCCA6" gate="G$1" x="81.28" y="264.16"/>
+<instance part="CN1" gate="G$1" x="175.26" y="180.34" rot="R180"/>
+<instance part="GND29" gate="G$1" x="180.34" y="175.26"/>
 </instances>
 <busses>
@@
 <pinref part="GND28" gate="G$1" pin="GND"/>
 </segment>
+<segment>
+<pinref part="CN1" gate="G$1" pin="P$1"/>
+<pinref part="GND29" gate="G$1" pin="GND"/>
+</segment>
 </net>
 <net name="VCC" class="0">
@@
 </segment>
 <segment>
-<pinref part="U1" gate="G$1" pin="PA6"/>
-<wire x1="223.52" y1="180.34" x2="220.98" y2="180.34" width="0.1524" layer="91"/>
-<label x="210.82" y="180.34" size="1.778" layer="95"/>
+<pinref part="U1" gate="G$1" pin="PC9"/>
+<wire x1="259.08" y1="147.32" x2="264.16" y2="147.32" width="0.1524" layer="91"/>
+<label x="264.16" y="147.32" size="1.778" layer="95"/>
 </segment>
 </net>
@@
 </segment>
 </net>
+<net name="N$12" class="0">
+<segment>
+<pinref part="U1" gate="G$1" pin="PA6"/>
+<pinref part="CN1" gate="G$1" pin="P$2"/>
+<wire x1="223.52" y1="180.34" x2="180.34" y2="180.34" width="0.1524" layer="91"/>
+</segment>
+</net>
