File: cad/gpi-ctl.sch (EAGLE design)
At the start: 101 parts, among them CN1 HEADER-1X2.4, CN2 MICROSDPLAIN, CN3 1X4-BIG, J4 1X4-BIG, SW1 SWITCHGT12-THOLE, SW2 SWITCHKMR211, SW3 SWITCHKMR211, U1 STM32F4/64, U2 ACS711, U3 ULN2003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

Commit message: lmp current sense
Parts:
- added C41: 1u, jaw:C0603
- added C42: .1u, jaw:C0603
- added R14: .01, jaw:R0603
- U2: value ACS711 -> LMP8640; device jaw:ACS711 -> jaw:LMP8640
Connections:
- removed net N$32: J2.P$7
- removed net N$45: J2.P$8
- removed net N$49: J3.P$8
- removed net N$53: J3.P$7
- net GND: now also C41.P$2, C42.P$2, J2.P$7, J2.P$8, J3.P$7, J3.P$8
- net VCC: no longer C25.P$1, C39.P$1, U2.VCC, U5.V
- net VCCA: now also C25.P$1, C39.P$1, C41.P$1, C42.P$1, U2.VCC, U5.V
- net VCCM: now also R14.P$1, U2.IN-; no longer U2.IP-
- net VIN: now also R14.P$2, U2.IN+; no longer U2.IP+
Other:
- moved on the sheet: C25

Commit message: filter
Parts:
- added C43: (no value), jaw:C0603
- added R21: (no value), jaw:R0603
Connections:
- new net N$18: R21.P$1, U2.VOUT
- net ADC12I: now also C43.P$1, R21.P$2; no longer U2.VOUT
- net GND: now also C43.P$2
Changed lines of the file:
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@@
 <part name="VCCA8" library="jaw" deviceset="PWR-VCCA" device=""/>
 <part name="C42" library="jaw" deviceset="C" device="0603" value=".1u"/>
+<part name="R21" library="jaw" deviceset="R" device="0603"/>
+<part name="C43" library="jaw" deviceset="C" device="0603"/>
 </parts>
 <sheets>
@@
 <instance part="LED3" gate="G$1" x="144.78" y="124.46"/>
 <instance part="C25" gate="G$1" x="78.74" y="91.44"/>
-<instance part="GND11" gate="G$1" x="78.74" y="81.28"/>
+<instance part="GND11" gate="G$1" x="78.74" y="71.12"/>
 <instance part="R16" gate="G$1" x="289.56" y="53.34"/>
 <instance part="R17" gate="G$1" x="279.4" y="50.8"/>
@@
 <instance part="VCCA8" gate="G$1" x="78.74" y="101.6"/>
 <instance part="C42" gate="G$1" x="35.56" y="223.52"/>
+<instance part="R21" gate="G$1" x="68.58" y="91.44"/>
+<instance part="C43" gate="G$1" x="73.66" y="76.2"/>
 </instances>
 <busses>
@@
 <wire x1="78.74" y1="88.9" x2="78.74" y2="86.36" width="0.1524" layer="91"/>
 <pinref part="U2" gate="G$1" pin="GND"/>
-<wire x1="78.74" y1="86.36" x2="78.74" y2="83.82" width="0.1524" layer="91"/>
+<wire x1="78.74" y1="86.36" x2="78.74" y2="73.66" width="0.1524" layer="91"/>
 <wire x1="63.5" y1="86.36" x2="78.74" y2="86.36" width="0.1524" layer="91"/>
 <junction x="78.74" y="86.36"/>
+<pinref part="C43" gate="G$1" pin="P$2"/>
+<wire x1="73.66" y1="73.66" x2="78.74" y2="73.66" width="0.1524" layer="91"/>
+<junction x="78.74" y="73.66"/>
 </segment>
 <segment>
@@
 </segment>
 <segment>
-<pinref part="U2" gate="G$1" pin="VOUT"/>
-<wire x1="63.5" y1="91.44" x2="68.58" y2="91.44" width="0.1524" layer="91"/>
-<label x="66.04" y="91.44" size="1.778" layer="95"/>
+<pinref part="R21" gate="G$1" pin="P$2"/>
+<pinref part="C43" gate="G$1" pin="P$1"/>
+<wire x1="73.66" y1="91.44" x2="73.66" y2="81.28" width="0.1524" layer="91"/>
+<wire x1="73.66" y1="81.28" x2="93.98" y2="81.28" width="0.1524" layer="91"/>
+<junction x="73.66" y="81.28"/>
+<label x="88.9" y="81.28" size="1.778" layer="95"/>
 </segment>
 </net>
@@
 </segment>
 </net>
+<net name="N$18" class="0">
+<segment>
+<pinref part="U2" gate="G$1" pin="VOUT"/>
+<pinref part="R21" gate="G$1" pin="P$1"/>
+</segment>
+</net>

Commit message: output filter
Parts:
- added C44: .1u 12V, jaw:C0603
- C1: value 10u 25V -> 10u 12V
- R14: device jaw:R0603 -> jaw:R0805
- renumbered VREG2 to U6
Connections:
- net ADC1: now also J3.P$1; no longer J2.P$1
- net ADC2: now also J3.P$2; no longer J2.P$2
- net ADC3: now also J3.P$3; no longer J2.P$3
- net ADC4: now also J3.P$4; no longer J2.P$4
- net ADC5: now also J3.P$5; no longer J2.P$5
- net ADC6: now also J3.P$6; no longer J2.P$6
- net GND: now also C44.P$2
- net IOG11: now also J2.P$3; no longer J3.P$3
- net IOG11N: now also J2.P$4; no longer J3.P$4
- net IOG12: now also J2.P$5; no longer J3.P$5
- net IOG12N: now also J2.P$6; no longer J3.P$6
- net IOG83: now also J2.P$1; no longer J3.P$1
- net IOG83N: now also J2.P$2; no longer J3.P$2
- net VCCM: now also C44.P$1
Other:
- moved on the sheet: J2, J3
Changed lines of the file:
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@@
 <part name="VCC14" library="jaw" deviceset="PWR-VCC" device=""/>
 <part name="VREG1" library="jaw" deviceset="REGULATOR" device="ROF" value=" ROF-78E3.3-0.5"/>
-<part name="C1" library="jaw" deviceset="C" device="0603" value="10u 25V"/>
+<part name="C1" library="jaw" deviceset="C" device="0603" value="10u 12V"/>
 <part name="C2" library="jaw" deviceset="C" device="1210" value="100u"/>
 <part name="C3" library="jaw" deviceset="C" device="0603" value="1u"/>
@@
 <part name="VCCM7" library="jaw" deviceset="PWR-VCCM" device=""/>
 <part name="J1" library="jaw" deviceset="HEADER-2X4" device=""/>
+<part name="J3" library="jaw" deviceset="HEADER-2X4" device=""/>
 <part name="J2" library="jaw" deviceset="HEADER-2X4" device=""/>
-<part name="J3" library="jaw" deviceset="HEADER-2X4" device=""/>
 <part name="R9" library="jaw" deviceset="R" device="0603" value="470"/>
 <part name="R11" library="jaw" deviceset="R" device="0603" value="1k"/>
@@
 <part name="C35" library="jaw" deviceset="C" device="0603" value=".1u"/>
 <part name="U$1" library="jaw" deviceset="ROBOTMAN-LOGO" device=""/>
-<part name="VREG2" library="jaw" deviceset="MCP1824" device=""/>
+<part name="U6" library="jaw" deviceset="MCP1824" device=""/>
 <part name="GND20" library="jaw" deviceset="PWR-GND" device=""/>
 <part name="VCC12" library="jaw" deviceset="PWR-VCC" device=""/>
@@
 <part name="GND33" library="jaw" deviceset="PWR-GND" device=""/>
 <part name="U2" library="jaw" deviceset="LMP8640" device=""/>
-<part name="R14" library="jaw" deviceset="R" device="0603" value=".01"/>
+<part name="R14" library="jaw" deviceset="R" device="0805" value=".01"/>
 <part name="C41" library="jaw" deviceset="C" device="0603" value="1u"/>
 <part name="VCCA7" library="jaw" deviceset="PWR-VCCA" device=""/>
@@
 <part name="R21" library="jaw" deviceset="R" device="0603"/>
 <part name="C43" library="jaw" deviceset="C" device="0603"/>
+<part name="C44" library="jaw" deviceset="C" device="0603" value=".1u 12V"/>
+<part name="GND12" library="jaw" deviceset="PWR-GND" device=""/>
+<part name="VCCM3" library="jaw" deviceset="PWR-VCCM" device=""/>
 </parts>
 <sheets>
@@
 <instance part="VCCM7" gate="G$1" x="381" y="162.56"/>
 <instance part="J1" gate="A" x="358.14" y="154.94"/>
-<instance part="J2" gate="A" x="358.14" y="139.7"/>
-<instance part="J3" gate="A" x="358.14" y="124.46"/>
+<instance part="J3" gate="A" x="358.14" y="139.7"/>
+<instance part="J2" gate="A" x="358.14" y="124.46"/>
 <instance part="R9" gate="G$1" x="114.3" y="132.08" rot="R90"/>
 <instance part="R11" gate="G$1" x="129.54" y="132.08" rot="R90"/>
@@
 <instance part="C35" gate="G$1" x="27.94" y="251.46"/>
 <instance part="U$1" gate="G$1" x="314.96" y="7.62"/>
-<instance part="VREG2" gate="G$1" x="350.52" y="73.66"/>
+<instance part="U6" gate="G$1" x="350.52" y="73.66"/>
 <instance part="GND20" gate="G$1" x="350.52" y="60.96"/>
 <instance part="VCC12" gate="G$1" x="373.38" y="78.74"/>
@@
 <instance part="R21" gate="G$1" x="68.58" y="91.44"/>
 <instance part="C43" gate="G$1" x="73.66" y="76.2"/>
+<instance part="C44" gate="G$1" x="60.96" y="223.52"/>
+<instance part="GND12" gate="G$1" x="60.96" y="218.44"/>
+<instance part="VCCM3" gate="G$1" x="60.96" y="231.14"/>
 </instances>
 <busses>
@@
 </segment>
 <segment>
-<pinref part="VREG2" gate="G$1" pin="GND"/>
+<pinref part="U6" gate="G$1" pin="GND"/>
 <pinref part="GND20" gate="G$1" pin="GND"/>
 <wire x1="350.52" y1="63.5" x2="350.52" y2="66.04" width="0.1524" layer="91"/>
@@
 </segment>
 <segment>
-<pinref part="J3" gate="A" pin="P$7"/>
+<pinref part="J2" gate="A" pin="P$7"/>
 <wire x1="355.6" y1="121.92" x2="350.52" y2="121.92" width="0.1524" layer="91"/>
 <pinref part="GND30" gate="G$1" pin="GND"/>
 </segment>
 <segment>
-<pinref part="J3" gate="A" pin="P$8"/>
+<pinref part="J2" gate="A" pin="P$8"/>
 <wire x1="363.22" y1="121.92" x2="373.38" y2="121.92" width="0.1524" layer="91"/>
 <pinref part="GND31" gate="G$1" pin="GND"/>
 </segment>
 <segment>
-<pinref part="J2" gate="A" pin="P$8"/>
+<pinref part="J3" gate="A" pin="P$8"/>
 <wire x1="363.22" y1="137.16" x2="373.38" y2="137.16" width="0.1524" layer="91"/>
 <pinref part="GND32" gate="G$1" pin="GND"/>
@@
 </segment>
 <segment>
-<pinref part="J2" gate="A" pin="P$7"/>
+<pinref part="J3" gate="A" pin="P$7"/>
 <wire x1="355.6" y1="137.16" x2="350.52" y2="137.16" width="0.1524" layer="91"/>
 <pinref part="GND33" gate="G$1" pin="GND"/>
 <wire x1="350.52" y1="137.16" x2="335.28" y2="137.16" width="0.1524" layer="91"/>
+</segment>
+<segment>
+<pinref part="C44" gate="G$1" pin="P$2"/>
+<pinref part="GND12" gate="G$1" pin="GND"/>
 </segment>
 </net>
@@
 <pinref part="VCC12" gate="G$1" pin="VCC"/>
 <pinref part="C36" gate="G$1" pin="P$1"/>
-<pinref part="VREG2" gate="G$1" pin="VOUT"/>
+<pinref part="U6" gate="G$1" pin="VOUT"/>
 <wire x1="365.76" y1="76.2" x2="373.38" y2="76.2" width="0.1524" layer="91"/>
 <junction x="373.38" y="76.2"/>
@@
 <junction x="373.38" y="160.02"/>
 </segment>
+<segment>
+<pinref part="C44" gate="G$1" pin="P$1"/>
+<pinref part="VCCM3" gate="G$1" pin="VCCM"/>
+</segment>
 </net>
 <net name="N$3" class="0">
@@
 <net name="ADC2" class="0">
 <segment>
-<pinref part="J2" gate="A" pin="P$2"/>
+<pinref part="J3" gate="A" pin="P$2"/>
 <wire x1="363.22" y1="144.78" x2="373.38" y2="144.78" width="0.1524" layer="91"/>
 <label x="373.38" y="144.78" size="1.778" layer="95"/>
@@
 <net name="ADC3" class="0">
 <segment>
-<pinref part="J2" gate="A" pin="P$3"/>
+<pinref part="J3" gate="A" pin="P$3"/>
 <wire x1="355.6" y1="142.24" x2="350.52" y2="142.24" width="0.1524" layer="91"/>
 <label x="345.44" y="142.24" size="1.778" layer="95"/>
@@
 <net name="ADC1" class="0">
 <segment>
-<pinref part="J2" gate="A" pin="P$1"/>
+<pinref part="J3" gate="A" pin="P$1"/>
 <wire x1="355.6" y1="144.78" x2="350.52" y2="144.78" width="0.1524" layer="91"/>
 <label x="345.44" y="144.78" size="1.778" layer="95"/>
@@
 <net name="ADC4" class="0">
 <segment>
-<pinref part="J2" gate="A" pin="P$4"/>
+<pinref part="J3" gate="A" pin="P$4"/>
 <wire x1="363.22" y1="142.24" x2="373.38" y2="142.24" width="0.1524" layer="91"/>
 <label x="373.38" y="142.24" size="1.778" layer="95"/>
@@
 <net name="ADC5" class="0">
 <segment>
-<pinref part="J2" gate="A" pin="P$5"/>
+<pinref part="J3" gate="A" pin="P$5"/>
 <wire x1="355.6" y1="139.7" x2="350.52" y2="139.7" width="0.1524" layer="91"/>
 <label x="345.44" y="139.7" size="1.778" layer="95"/>
@@
 <net name="ADC6" class="0">
 <segment>
-<pinref part="J2" gate="A" pin="P$6"/>
+<pinref part="J3" gate="A" pin="P$6"/>
 <wire x1="363.22" y1="139.7" x2="373.38" y2="139.7" width="0.1524" layer="91"/>
 <label x="373.38" y="139.7" size="1.778" layer="95"/>
@@
 </segment>
 <segment>
-<pinref part="J3" gate="A" pin="P$6"/>
+<pinref part="J2" gate="A" pin="P$6"/>
 <wire x1="363.22" y1="124.46" x2="373.38" y2="124.46" width="0.1524" layer="91"/>
 <label x="373.38" y="124.46" size="1.778" layer="95"/>
@@
 </segment>
 <segment>
-<pinref part="J3" gate="A" pin="P$2"/>
+<pinref part="J2" gate="A" pin="P$2"/>
 <wire x1="363.22" y1="129.54" x2="373.38" y2="129.54" width="0.1524" layer="91"/>
 <label x="373.38" y="129.54" size="1.778" layer="95"/>
@@
 </segment>
 <segment>
-<pinref part="J3" gate="A" pin="P$4"/>
+<pinref part="J2" gate="A" pin="P$4"/>
 <wire x1="363.22" y1="127" x2="373.38" y2="127" width="0.1524" layer="91"/>
 <label x="373.38" y="127" size="1.778" layer="95"/>
@@
 </segment>
 <segment>
-<pinref part="J3" gate="A" pin="P$3"/>
+<pinref part="J2" gate="A" pin="P$3"/>
 <wire x1="355.6" y1="127" x2="350.52" y2="127" width="0.1524" layer="91"/>
 <label x="342.9" y="127" size="1.778" layer="95"/>
@@
 </segment>
 <segment>
-<pinref part="J3" gate="A" pin="P$5"/>
+<pinref part="J2" gate="A" pin="P$5"/>
 <wire x1="355.6" y1="124.46" x2="350.52" y2="124.46" width="0.1524" layer="91"/>
 <label x="342.9" y="124.46" size="1.778" layer="95"/>
@@
 </segment>
 <segment>
-<pinref part="J3" gate="A" pin="P$1"/>
+<pinref part="J2" gate="A" pin="P$1"/>
 <wire x1="355.6" y1="129.54" x2="350.52" y2="129.54" width="0.1524" layer="91"/>
 <label x="342.9" y="129.54" size="1.778" layer="95"/>
@@
 <net name="N$8" class="0">
 <segment>
-<pinref part="VREG2" gate="G$1" pin="VIN"/>
+<pinref part="U6" gate="G$1" pin="VIN"/>
 <pinref part="D2" gate="G$1" pin="C"/>
 <wire x1="335.28" y1="76.2" x2="332.74" y2="76.2" width="0.1524" layer="91"/>
-<pinref part="VREG2" gate="G$1" pin="NSHTDN"/>
+<pinref part="U6" gate="G$1" pin="NSHTDN"/>
 <wire x1="332.74" y1="76.2" x2="304.8" y2="76.2" width="0.1524" layer="91"/>
 <wire x1="335.28" y1="73.66" x2="332.74" y2="73.66" width="0.1524" layer="91"/>

Commit message: tweak
Parts:
- C43: value (none) -> .1u
- R21: value (none) -> 100
Changed lines of the file:
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@@
 <part name="VCCA8" library="jaw" deviceset="PWR-VCCA" device=""/>
 <part name="C42" library="jaw" deviceset="C" device="0603" value=".1u"/>
-<part name="R21" library="jaw" deviceset="R" device="0603"/>
-<part name="C43" library="jaw" deviceset="C" device="0603"/>
+<part name="R21" library="jaw" deviceset="R" device="0603" value="100"/>
+<part name="C43" library="jaw" deviceset="C" device="0603" value=".1u"/>
 <part name="C44" library="jaw" deviceset="C" device="0603" value=".1u 12V"/>
 <part name="GND12" library="jaw" deviceset="PWR-GND" device=""/>

Commit message: bigger cap
Parts:
- C10, C17: value .001u -> .1u
Changed lines of the file:
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@@
 <part name="D7" library="jaw" deviceset="ZENER" device="" value="4v"/>
 <part name="D8" library="jaw" deviceset="ZENER" device="" value="4v"/>
-<part name="C10" library="jaw" deviceset="C" device="0603" value=".001u"/>
+<part name="C10" library="jaw" deviceset="C" device="0603" value=".1u"/>
 <part name="C11" library="jaw" deviceset="C" device="0603" value=".1u"/>
 <part name="C12" library="jaw" deviceset="C" device="0603" value=".1u"/>
 <part name="C13" library="jaw" deviceset="C" device="0603" value="1u"/>
 <part name="C14" library="jaw" deviceset="C" device="0603" value="1u"/>
-<part name="C17" library="jaw" deviceset="C" device="0603" value=".001u"/>
+<part name="C17" library="jaw" deviceset="C" device="0603" value=".1u"/>
 <part name="R1" library="jaw" deviceset="R" device="0603" value="100"/>
 <part name="R2" library="jaw" deviceset="R" device="0603" value="100"/>

Commit message: caps
Parts:
- C12: value .1u -> .01u
Changed lines of the file:
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@@
 <part name="C10" library="jaw" deviceset="C" device="0603" value=".1u"/>
 <part name="C11" library="jaw" deviceset="C" device="0603" value=".1u"/>
-<part name="C12" library="jaw" deviceset="C" device="0603" value=".1u"/>
+<part name="C12" library="jaw" deviceset="C" device="0603" value=".01u"/>
 <part name="C13" library="jaw" deviceset="C" device="0603" value="1u"/>
 <part name="C14" library="jaw" deviceset="C" device="0603" value="1u"/>

Commit message: comments
Other:
- note added: "OLED display"
- note added: "TXCO"
- note added: "USB/serial - diag + programming"
- note added: "diag sync out (to trigger scope)"
- note added: "diag user input"
- note added: "input voltage sense (resistor divider on other board)"
- note added: "seperate/smaller reg for USB power in"
- note added: "to power board"
- note added: "voltage+current sense low-pass"
- note removed: "M471-OLED display"
- note removed: "Sync Out"
- moved on the sheet: C29, C36, C8, D2, J1, J2, J3, J4, LED5, LED6, R10, R16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

Commit message: pdfs, comments
Other:
- note added: "power inverter - control board little box challenge"
Changed lines of the file:
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@@
 <setting verticaltext="up"/>
 </settings>
-<grid distance="0.1" unitdist="inch" unit="inch" style="lines" multiple="1" display="yes" altdistance="0.01" altunitdist="inch" altunit="inch"/>
+<grid distance="0.1" unitdist="inch" unit="inch" style="lines" multiple="1" display="no" altdistance="0.01" altunitdist="inch" altunit="inch"/>
 <layers>
 <layer number="1" name="Top" color="4" fill="1" visible="no" active="no"/>
@@
 <wire x1="325.12" y1="78.74" x2="325.12" y2="86.36" width="0.508" layer="97"/>
 <text x="218.44" y="71.12" size="1.778" layer="97">USB/serial - diag + programming</text>
+<text x="330.2" y="25.4" size="2.54" layer="94" ratio="10">power inverter - control board
+little box challenge</text>
 </plain>
 <instances>
