File: cad/gpi-ctl.sch (EAGLE design)
At the start: 107 parts, among them CN1 HEADER-1X2.4, CN2 MICROSDPLAIN, CN3 1X4-BIG, J4 1X4-BIG, SW1 SWITCHGT12-THOLE, SW2 SWITCHKMR211, SW3 SWITCHKMR211, U1 STM32F4/64, U2 LMP8640, U3 ULN2003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

Commit message: revert opamp, tweak
Parts:
- removed C8: 2.2u, jaw:C0603
- removed LED5: GREEN, jaw:LED
- removed LED6: ORANGE, jaw:LED
- removed R10: 270, jaw:R0603
- removed R23: 560, jaw:R0603
- removed U8: IC_FT230X-SSOP-16, dp_devices:IC_FT230X-SSOP-16
Connections:
- removed net N$20: R17.P$1, U8.USB+
- removed net N$25: R23.P$1, U8.CBUS2
- removed net N$26: R10.P$1, U8.CBUS1
- removed net N$38: LED5.C, R10.P$2
- removed net N$41: LED6.C, R23.P$2
- removed net N$42: R16.P$1, U8.USB-
- removed net USB3V3: C8.P$1, LED5.A, LED6.A, U8.!RESET, U8.3V3OUT, U8.VCCIO
- new net USBDM: R16.P$1, U1.PA11
- new net USBDP: R17.P$1, U1.PA12
- net GND: no longer C8.P$2, U8.GND@1, U8.GND@2
- net IOCARD: now also U1.PA13; no longer U1.PA11
- net RX: no longer U8.TXD
- net TX: no longer U8.RXD
- net VBUS: no longer U8.VCC
Other:
- moved on the sheet: C29, D2
Changed lines of the file:
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@@
 <?xml version="1.0" encoding="utf-8"?>
 <!DOCTYPE eagle SYSTEM "eagle.dtd">
-<eagle version="7.2.0">
+<eagle version="7.5.0">
 <drawing>
 <settings>
@@
 <part name="GND24" library="jaw" deviceset="PWR-GND" device=""/>
 <part name="VCC20" library="jaw" deviceset="PWR-VCC" device=""/>
-<part name="U8" library="dp_devices" deviceset="IC_FT230X" device="-SSOP-16"/>
-<part name="GND8" library="jaw" deviceset="PWR-GND" device=""/>
 <part name="GND37" library="jaw" deviceset="PWR-GND" device=""/>
-<part name="C8" library="jaw" deviceset="C" device="0603" value="2.2u"/>
-<part name="GND44" library="jaw" deviceset="PWR-GND" device=""/>
-<part name="R10" library="jaw" deviceset="R" device="0603" value="270"/>
-<part name="R23" library="jaw" deviceset="R" device="0603" value="560"/>
-<part name="LED5" library="jaw" deviceset="LED" device="" value="GREEN"/>
-<part name="LED6" library="jaw" deviceset="LED" device="" value="ORANGE"/>
 <part name="C29" library="jaw" deviceset="C" device="0603" value="1u"/>
 <part name="GND46" library="jaw" deviceset="PWR-GND" device=""/>
@@
 <instance part="GND24" gate="G$1" x="218.44" y="96.52"/>
 <instance part="VCC20" gate="G$1" x="190.5" y="109.22"/>
-<instance part="U8" gate="IC" x="231.14" y="33.02"/>
-<instance part="GND8" gate="G$1" x="231.14" y="12.7"/>
 <instance part="GND37" gate="G$1" x="292.1" y="12.7"/>
-<instance part="C8" gate="G$1" x="251.46" y="20.32"/>
-<instance part="GND44" gate="G$1" x="251.46" y="12.7"/>
-<instance part="R10" gate="G$1" x="205.74" y="27.94" rot="R180"/>
-<instance part="R23" gate="G$1" x="205.74" y="20.32" rot="R180"/>
-<instance part="LED5" gate="G$1" x="195.58" y="27.94"/>
-<instance part="LED6" gate="G$1" x="195.58" y="20.32"/>
-<instance part="C29" gate="G$1" x="281.94" y="53.34"/>
-<instance part="GND46" gate="G$1" x="281.94" y="48.26"/>
-<instance part="D2" gate="G$1" x="289.56" y="58.42"/>
+<instance part="C29" gate="G$1" x="279.4" y="63.5"/>
+<instance part="GND46" gate="G$1" x="279.4" y="55.88"/>
+<instance part="D2" gate="G$1" x="287.02" y="68.58"/>
 <instance part="USB1" gate="USB" x="297.18" y="35.56" rot="MR0"/>
 <instance part="NY1" gate="G$1" x="340.36" y="248.92"/>
@@
 </segment>
 <segment>
-<pinref part="U8" gate="IC" pin="GND@1"/>
-<pinref part="GND8" gate="G$1" pin="GND"/>
-<wire x1="231.14" y1="15.24" x2="231.14" y2="17.78" width="0.1524" layer="91"/>
-<pinref part="U8" gate="IC" pin="GND@2"/>
-<wire x1="233.68" y1="17.78" x2="231.14" y2="17.78" width="0.1524" layer="91"/>
-<junction x="231.14" y="17.78"/>
-</segment>
-<segment>
-<pinref part="C8" gate="G$1" pin="P$2"/>
-<pinref part="GND44" gate="G$1" pin="GND"/>
-<wire x1="251.46" y1="15.24" x2="251.46" y2="17.78" width="0.1524" layer="91"/>
-</segment>
-<segment>
 <pinref part="C29" gate="G$1" pin="P$2"/>
 <pinref part="GND46" gate="G$1" pin="GND"/>
+<wire x1="279.4" y1="60.96" x2="279.4" y2="58.42" width="0.1524" layer="91"/>
 </segment>
 <segment>
@@
 <label x="261.62" y="144.78" size="1.778" layer="95"/>
 </segment>
-<segment>
-<pinref part="U8" gate="IC" pin="RXD"/>
-<wire x1="215.9" y1="40.64" x2="213.36" y2="40.64" width="0.1524" layer="91"/>
-<label x="210.82" y="40.64" size="1.778" layer="95"/>
-</segment>
 </net>
 <net name="RX" class="0">
@@
 <label x="261.62" y="142.24" size="1.778" layer="95"/>
 </segment>
-<segment>
-<pinref part="U8" gate="IC" pin="TXD"/>
-<wire x1="215.9" y1="43.18" x2="213.36" y2="43.18" width="0.1524" layer="91"/>
-<label x="210.82" y="43.18" size="1.778" layer="95"/>
-</segment>
 </net>
 <net name="DPYDC" class="0">
@@
 </segment>
 </net>
-<net name="N$20" class="0">
-<segment>
-<pinref part="U8" gate="IC" pin="USB+"/>
-<wire x1="248.92" y1="33.02" x2="256.54" y2="33.02" width="0.1524" layer="91"/>
-<pinref part="R17" gate="G$1" pin="P$1"/>
-<wire x1="256.54" y1="33.02" x2="261.62" y2="33.02" width="0.1524" layer="91"/>
-</segment>
-</net>
-<net name="N$26" class="0">
-<segment>
-<pinref part="R10" gate="G$1" pin="P$1"/>
-<pinref part="U8" gate="IC" pin="CBUS1"/>
-<wire x1="210.82" y1="27.94" x2="215.9" y2="27.94" width="0.1524" layer="91"/>
-</segment>
-</net>
-<net name="N$25" class="0">
-<segment>
-<pinref part="R23" gate="G$1" pin="P$1"/>
-<pinref part="U8" gate="IC" pin="CBUS2"/>
-<wire x1="210.82" y1="20.32" x2="210.82" y2="25.4" width="0.1524" layer="91"/>
-<wire x1="210.82" y1="25.4" x2="215.9" y2="25.4" width="0.1524" layer="91"/>
-</segment>
-</net>
-<net name="USB3V3" class="0">
-<segment>
-<pinref part="U8" gate="IC" pin="VCCIO"/>
-<wire x1="233.68" y1="48.26" x2="233.68" y2="50.8" width="0.1524" layer="91"/>
-<wire x1="233.68" y1="50.8" x2="251.46" y2="50.8" width="0.1524" layer="91"/>
-<wire x1="251.46" y1="50.8" x2="251.46" y2="40.64" width="0.1524" layer="91"/>
-<pinref part="U8" gate="IC" pin="3V3OUT"/>
-<wire x1="251.46" y1="40.64" x2="248.92" y2="40.64" width="0.1524" layer="91"/>
-<wire x1="251.46" y1="40.64" x2="251.46" y2="25.4" width="0.1524" layer="91"/>
-<junction x="251.46" y="40.64"/>
-<pinref part="U8" gate="IC" pin="!RESET"/>
-<wire x1="251.46" y1="25.4" x2="248.92" y2="25.4" width="0.1524" layer="91"/>
-<pinref part="C8" gate="G$1" pin="P$1"/>
-<junction x="251.46" y="25.4"/>
-<pinref part="LED6" gate="G$1" pin="A"/>
-<pinref part="LED5" gate="G$1" pin="A"/>
-<wire x1="190.5" y1="20.32" x2="190.5" y2="27.94" width="0.1524" layer="91"/>
-<wire x1="190.5" y1="27.94" x2="190.5" y2="50.8" width="0.1524" layer="91"/>
-<wire x1="190.5" y1="50.8" x2="233.68" y2="50.8" width="0.1524" layer="91"/>
-<junction x="190.5" y="27.94"/>
-<junction x="233.68" y="50.8"/>
-</segment>
-</net>
-<net name="N$38" class="0">
-<segment>
-<pinref part="R10" gate="G$1" pin="P$2"/>
-<pinref part="LED5" gate="G$1" pin="C"/>
-</segment>
-</net>
-<net name="N$41" class="0">
-<segment>
-<pinref part="LED6" gate="G$1" pin="C"/>
-<pinref part="R23" gate="G$1" pin="P$2"/>
-</segment>
-</net>
 <net name="VBUS" class="0">
 <segment>
-<pinref part="U8" gate="IC" pin="VCC"/>
-<wire x1="228.6" y1="48.26" x2="228.6" y2="53.34" width="0.1524" layer="91"/>
-<wire x1="228.6" y1="53.34" x2="256.54" y2="53.34" width="0.1524" layer="91"/>
-<wire x1="256.54" y1="53.34" x2="256.54" y2="38.1" width="0.1524" layer="91"/>
-<wire x1="256.54" y1="38.1" x2="266.7" y2="38.1" width="0.1524" layer="91"/>
 <wire x1="266.7" y1="38.1" x2="271.78" y2="38.1" width="0.1524" layer="91"/>
-<wire x1="266.7" y1="38.1" x2="266.7" y2="58.42" width="0.1524" layer="91"/>
-<wire x1="266.7" y1="58.42" x2="281.94" y2="58.42" width="0.1524" layer="91"/>
-<junction x="266.7" y="38.1"/>
+<wire x1="266.7" y1="38.1" x2="266.7" y2="68.58" width="0.1524" layer="91"/>
+<wire x1="266.7" y1="68.58" x2="279.4" y2="68.58" width="0.1524" layer="91"/>
 <pinref part="C29" gate="G$1" pin="P$1"/>
 <pinref part="D2" gate="G$1" pin="A"/>
-<wire x1="281.94" y1="58.42" x2="287.02" y2="58.42" width="0.1524" layer="91"/>
-<junction x="281.94" y="58.42"/>
+<wire x1="279.4" y1="68.58" x2="284.48" y2="68.58" width="0.1524" layer="91"/>
+<junction x="279.4" y="68.58"/>
 <pinref part="USB1" gate="USB" pin="VUSB"/>
 <wire x1="271.78" y1="38.1" x2="292.1" y2="38.1" width="0.1524" layer="91"/>
-</segment>
-</net>
-<net name="N$42" class="0">
-<segment>
-<pinref part="U8" gate="IC" pin="USB-"/>
-<wire x1="248.92" y1="35.56" x2="256.54" y2="35.56" width="0.1524" layer="91"/>
-<pinref part="R16" gate="G$1" pin="P$1"/>
-<wire x1="271.78" y1="35.56" x2="256.54" y2="35.56" width="0.1524" layer="91"/>
 </segment>
 </net>
@@
 <net name="IOCARD" class="0">
 <segment>
-<pinref part="U1" gate="G$1" pin="PA11"/>
-<wire x1="259.08" y1="187.96" x2="264.16" y2="187.96" width="0.1524" layer="91"/>
-<label x="264.16" y="187.96" size="1.778" layer="95"/>
-</segment>
-<segment>
 <pinref part="CN2" gate="G$1" pin="SW2"/>
 <pinref part="R18" gate="G$1" pin="P$1"/>
@@
 <wire x1="289.56" y1="96.52" x2="302.26" y2="96.52" width="0.1524" layer="91"/>
 <label x="297.18" y="96.52" size="1.778" layer="95"/>
+</segment>
+<segment>
+<pinref part="U1" gate="G$1" pin="PA13"/>
+<wire x1="259.08" y1="182.88" x2="264.16" y2="182.88" width="0.1524" layer="91"/>
+<label x="264.16" y="182.88" size="1.778" layer="95" ratio="10"/>
 </segment>
 </net>
@@
 <pinref part="U6" gate="G$1" pin="NSHTDN"/>
 <wire x1="332.74" y1="68.58" x2="292.1" y2="68.58" width="0.1524" layer="91"/>
-<wire x1="292.1" y1="68.58" x2="292.1" y2="58.42" width="0.1524" layer="91"/>
+<wire x1="292.1" y1="68.58" x2="289.56" y2="68.58" width="0.1524" layer="91"/>
 <wire x1="335.28" y1="66.04" x2="332.74" y2="66.04" width="0.1524" layer="91"/>
 <wire x1="332.74" y1="66.04" x2="332.74" y2="68.58" width="0.1524" layer="91"/>
@@
 </segment>
 </net>
+<net name="USBDM" class="0">
+<segment>
+<pinref part="U1" gate="G$1" pin="PA11"/>
+<wire x1="259.08" y1="187.96" x2="264.16" y2="187.96" width="0.1524" layer="91"/>
+<label x="264.16" y="187.96" size="1.778" layer="95" ratio="10"/>
+</segment>
+<segment>
+<wire x1="248.92" y1="35.56" x2="256.54" y2="35.56" width="0.1524" layer="91"/>
+<pinref part="R16" gate="G$1" pin="P$1"/>
+<wire x1="271.78" y1="35.56" x2="256.54" y2="35.56" width="0.1524" layer="91"/>
+<label x="241.3" y="35.56" size="1.778" layer="95" ratio="10"/>
+</segment>
+</net>
+<net name="USBDP" class="0">
+<segment>
+<pinref part="U1" gate="G$1" pin="PA12"/>
+<wire x1="259.08" y1="185.42" x2="264.16" y2="185.42" width="0.1524" layer="91"/>
+<label x="264.16" y="185.42" size="1.778" layer="95" ratio="10"/>
+</segment>
+<segment>
+<wire x1="248.92" y1="33.02" x2="256.54" y2="33.02" width="0.1524" layer="91"/>
+<pinref part="R17" gate="G$1" pin="P$1"/>
+<wire x1="256.54" y1="33.02" x2="261.62" y2="33.02" width="0.1524" layer="91"/>
+<label x="241.3" y="33.02" size="1.778" layer="95" ratio="10"/>
+</segment>
+</net>
