File: cad/gpi-pwr.sch (EAGLE design)
At the start: 87 parts, among them CN1 HEADER-1X2, CN2 HEADER-3X1, CN3 HEADER-1X2.4, Q1 MOSFETTO247REV, Q3 MOSFETTO247REV, Q5 MOSFETTO247REV, Q6 MOSFETTO247REV, Q7 MOSFETTO247REV, Q8 MOSFETTO247REV, U1 ACS709, U2 ACS709, U3 ACPL-P346P346, U4 ACPL-P346P346, U5 ACPL-P346P346, U6 ACPL-P346P346, U7 ACPL-P346P346, U8 ACPL-P346P346

Commit message: tweak
Parts:
- added C26: .1u, jaw:C2220
- added R25: 1M, jaw:R1206
- C3: value .1u CER -> .1u
Connections:
- net GND: now also C26.P$2, R25.P$1
- net N$7: now also R25.P$2
- net V1KDC: now also C26.P$1
Changed lines of the file:
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@@
 <setting verticaltext="up"/>
 </settings>
-<grid distance="0.1" unitdist="inch" unit="inch" style="lines" multiple="1" display="yes" altdistance="0.01" altunitdist="inch" altunit="inch"/>
+<grid distance="0.1" unitdist="inch" unit="inch" style="lines" multiple="1" display="no" altdistance="0.01" altunitdist="inch" altunit="inch"/>
 <layers>
 <layer number="1" name="Top" color="4" fill="1" visible="no" active="no"/>
@@
 <part name="C1" library="jaw" deviceset="C" device="R46KI333000N1M" value=".33u"/>
 <part name="C2" library="jaw" deviceset="C" device="MKP1848S62010JY5F" value="20u"/>
-<part name="C3" library="jaw" deviceset="C" device="2220" value=".1u CER"/>
+<part name="C3" library="jaw" deviceset="C" device="2220" value=".1u"/>
 <part name="R1" library="jaw" deviceset="R" device="2512" value="1M 2kV"/>
 <part name="Q1" library="jaw" deviceset="MOSFET" device="TO247REV" value="MOSFETTO247REV"/>
@@
 <part name="U$6" library="jaw" deviceset="SYMBOL-WARNING" device=""/>
 <part name="U$7" library="jaw" deviceset="SYMBOL-WARNING" device=""/>
+<part name="C26" library="jaw" deviceset="C" device="2220" value=".1u"/>
+<part name="R25" library="jaw" deviceset="R" device="1206" value="1M"/>
 </parts>
 <sheets>
@@
 <instance part="U$6" gate="G$1" x="355.6" y="45.72"/>
 <instance part="U$7" gate="G$1" x="342.9" y="45.72"/>
+<instance part="C26" gate="G$1" x="132.08" y="86.36"/>
+<instance part="R25" gate="G$1" x="50.8" y="78.74" rot="R90"/>
 </instances>
 <busses>
@@
 <wire x1="20.32" y1="68.58" x2="45.72" y2="68.58" width="0.1524" layer="91"/>
 <junction x="45.72" y="68.58"/>
+<pinref part="R25" gate="G$1" pin="P$1"/>
+<wire x1="50.8" y1="73.66" x2="50.8" y2="68.58" width="0.1524" layer="91"/>
+<wire x1="50.8" y1="68.58" x2="45.72" y2="68.58" width="0.1524" layer="91"/>
 </segment>
 <segment>
@@
 <pinref part="C4" gate="G$1" pin="P$2"/>
 <wire x1="121.92" y1="83.82" x2="121.92" y2="78.74" width="0.1524" layer="91"/>
+<pinref part="C26" gate="G$1" pin="P$2"/>
+<wire x1="132.08" y1="83.82" x2="132.08" y2="78.74" width="0.1524" layer="91"/>
+<wire x1="132.08" y1="78.74" x2="127" y2="78.74" width="0.1524" layer="91"/>
+<junction x="127" y="78.74"/>
 </segment>
 <segment>
@@
 <junction x="215.9" y="104.14"/>
 <pinref part="R1" gate="G$1" pin="P$2"/>
-<wire x1="127" y1="96.52" x2="142.24" y2="96.52" width="0.1524" layer="91"/>
+<wire x1="127" y1="96.52" x2="132.08" y2="96.52" width="0.1524" layer="91"/>
 <pinref part="C3" gate="G$1" pin="P$1"/>
+<wire x1="132.08" y1="96.52" x2="142.24" y2="96.52" width="0.1524" layer="91"/>
 <wire x1="127" y1="91.44" x2="127" y2="96.52" width="0.1524" layer="91"/>
 <junction x="127" y="96.52"/>
@@
 <junction x="116.84" y="96.52"/>
 <label x="149.86" y="101.6" size="1.778" layer="95"/>
+<pinref part="C26" gate="G$1" pin="P$1"/>
+<wire x1="132.08" y1="91.44" x2="132.08" y2="96.52" width="0.1524" layer="91"/>
+<junction x="132.08" y="96.52"/>
 </segment>
 </net>
@@
 <wire x1="35.56" y1="101.6" x2="35.56" y2="96.52" width="0.1524" layer="91"/>
 <pinref part="L1" gate="G$1" pin="P$1"/>
-<wire x1="48.26" y1="96.52" x2="53.34" y2="96.52" width="0.1524" layer="91"/>
+<wire x1="48.26" y1="96.52" x2="50.8" y2="96.52" width="0.1524" layer="91"/>
+<wire x1="50.8" y1="96.52" x2="53.34" y2="96.52" width="0.1524" layer="91"/>
 <wire x1="35.56" y1="96.52" x2="40.64" y2="96.52" width="0.1524" layer="91"/>
 <pinref part="C1" gate="G$1" pin="P$1"/>
@@
 <wire x1="40.64" y1="71.12" x2="40.64" y2="96.52" width="0.1524" layer="91"/>
 <junction x="40.64" y="96.52"/>
-</segment>
-</net>
+<pinref part="R25" gate="G$1" pin="P$2"/>
+<wire x1="50.8" y1="83.82" x2="50.8" y2="96.52" width="0.1524" layer="91"/>
+<junction x="50.8" y="96.52"/>
+</segment>
+</net>

Commit message: better output filter
Connections:
- net GND: no longer C6.P$2, C7.P$1
- net N$15: now also C6.P$1
- net N$16: now also C6.P$2
- net N$24: now also C7.P$1; no longer C6.P$1
Other:
- moved on the sheet: C6, C7, L3, L4
Changed lines of the file:
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@@
 <instance part="Q7" gate="G$1" x="264.16" y="96.52"/>
 <instance part="Q8" gate="G$1" x="264.16" y="76.2"/>
-<instance part="L3" gate="G$1" x="317.5" y="99.06"/>
-<instance part="L4" gate="G$1" x="317.5" y="73.66"/>
-<instance part="C6" gate="G$1" x="327.66" y="93.98"/>
-<instance part="C7" gate="G$1" x="327.66" y="76.2"/>
+<instance part="L3" gate="G$1" x="304.8" y="99.06"/>
+<instance part="L4" gate="G$1" x="304.8" y="73.66"/>
+<instance part="C6" gate="G$1" x="294.64" y="86.36"/>
+<instance part="C7" gate="G$1" x="312.42" y="86.36"/>
 <instance part="R5" gate="G$1" x="142.24" y="76.2" rot="R90"/>
 <instance part="R10" gate="G$1" x="335.28" y="86.36" rot="R180"/>
@@
 </segment>
 <segment>
-<pinref part="C6" gate="G$1" pin="P$2"/>
-<pinref part="C7" gate="G$1" pin="P$1"/>
-<wire x1="327.66" y1="81.28" x2="327.66" y2="86.36" width="0.1524" layer="91"/>
 <pinref part="GND10" gate="G$1" pin="GND"/>
-<wire x1="327.66" y1="86.36" x2="327.66" y2="91.44" width="0.1524" layer="91"/>
 <wire x1="320.04" y1="86.36" x2="327.66" y2="86.36" width="0.1524" layer="91"/>
-<junction x="327.66" y="86.36"/>
 <pinref part="R10" gate="G$1" pin="P$2"/>
 <wire x1="330.2" y1="86.36" x2="327.66" y2="86.36" width="0.1524" layer="91"/>
@@
 <net name="N$24" class="0">
 <segment>
-<wire x1="327.66" y1="99.06" x2="358.14" y2="99.06" width="0.1524" layer="91"/>
 <wire x1="358.14" y1="99.06" x2="365.76" y2="99.06" width="0.1524" layer="91"/>
 <wire x1="365.76" y1="99.06" x2="365.76" y2="101.6" width="0.1524" layer="91"/>
@@
 <wire x1="358.14" y1="93.98" x2="358.14" y2="99.06" width="0.1524" layer="91"/>
 <junction x="358.14" y="99.06"/>
-<pinref part="C6" gate="G$1" pin="P$1"/>
 <pinref part="L3" gate="G$1" pin="P$2"/>
-<wire x1="325.12" y1="99.06" x2="327.66" y2="99.06" width="0.1524" layer="91"/>
-<junction x="327.66" y="99.06"/>
+<wire x1="312.42" y1="99.06" x2="358.14" y2="99.06" width="0.1524" layer="91"/>
+<pinref part="C7" gate="G$1" pin="P$1"/>
+<wire x1="312.42" y1="91.44" x2="312.42" y2="99.06" width="0.1524" layer="91"/>
+<junction x="312.42" y="99.06"/>
 </segment>
 </net>
@@
 <segment>
 <pinref part="CN2" gate="G$1" pin="3"/>
-<wire x1="327.66" y1="73.66" x2="358.14" y2="73.66" width="0.1524" layer="91"/>
 <wire x1="358.14" y1="73.66" x2="401.32" y2="73.66" width="0.1524" layer="91"/>
 <wire x1="401.32" y1="73.66" x2="408.94" y2="73.66" width="0.1524" layer="91"/>
@@
 <pinref part="C7" gate="G$1" pin="P$2"/>
 <pinref part="L4" gate="G$1" pin="P$2"/>
-<wire x1="325.12" y1="73.66" x2="327.66" y2="73.66" width="0.1524" layer="91"/>
-<junction x="327.66" y="73.66"/>
+<wire x1="312.42" y1="73.66" x2="312.42" y2="83.82" width="0.1524" layer="91"/>
 <pinref part="R3" gate="G$1" pin="P$1"/>
 <wire x1="401.32" y1="76.2" x2="401.32" y2="73.66" width="0.1524" layer="91"/>
 <junction x="401.32" y="73.66"/>
+<wire x1="312.42" y1="73.66" x2="358.14" y2="73.66" width="0.1524" layer="91"/>
+<junction x="312.42" y="73.66"/>
 </segment>
 </net>
@@
 <wire x1="215.9" y1="81.28" x2="215.9" y2="88.9" width="0.1524" layer="91"/>
 <wire x1="215.9" y1="88.9" x2="215.9" y2="91.44" width="0.1524" layer="91"/>
-<wire x1="215.9" y1="88.9" x2="307.34" y2="88.9" width="0.1524" layer="91"/>
-<wire x1="307.34" y1="88.9" x2="307.34" y2="99.06" width="0.1524" layer="91"/>
+<wire x1="215.9" y1="88.9" x2="287.02" y2="88.9" width="0.1524" layer="91"/>
+<wire x1="287.02" y1="88.9" x2="287.02" y2="99.06" width="0.1524" layer="91"/>
 <junction x="215.9" y="88.9"/>
-<wire x1="307.34" y1="99.06" x2="309.88" y2="99.06" width="0.1524" layer="91"/>
+<wire x1="287.02" y1="99.06" x2="294.64" y2="99.06" width="0.1524" layer="91"/>
 <pinref part="L3" gate="G$1" pin="P$1"/>
+<wire x1="294.64" y1="99.06" x2="297.18" y2="99.06" width="0.1524" layer="91"/>
 <wire x1="198.12" y1="116.84" x2="198.12" y2="88.9" width="0.1524" layer="91"/>
 <wire x1="198.12" y1="88.9" x2="215.9" y2="88.9" width="0.1524" layer="91"/>
 <junction x="198.12" y="116.84"/>
+<pinref part="C6" gate="G$1" pin="P$1"/>
+<wire x1="294.64" y1="91.44" x2="294.64" y2="99.06" width="0.1524" layer="91"/>
+<junction x="294.64" y="99.06"/>
 </segment>
 </net>
@@
 <wire x1="264.16" y1="81.28" x2="264.16" y2="83.82" width="0.1524" layer="91"/>
 <wire x1="264.16" y1="83.82" x2="264.16" y2="91.44" width="0.1524" layer="91"/>
-<wire x1="264.16" y1="83.82" x2="307.34" y2="83.82" width="0.1524" layer="91"/>
-<wire x1="307.34" y1="83.82" x2="307.34" y2="73.66" width="0.1524" layer="91"/>
+<wire x1="264.16" y1="83.82" x2="287.02" y2="83.82" width="0.1524" layer="91"/>
+<wire x1="287.02" y1="83.82" x2="287.02" y2="73.66" width="0.1524" layer="91"/>
 <junction x="264.16" y="83.82"/>
-<wire x1="307.34" y1="73.66" x2="309.88" y2="73.66" width="0.1524" layer="91"/>
+<wire x1="287.02" y1="73.66" x2="294.64" y2="73.66" width="0.1524" layer="91"/>
 <pinref part="L4" gate="G$1" pin="P$1"/>
+<wire x1="294.64" y1="73.66" x2="297.18" y2="73.66" width="0.1524" layer="91"/>
 <wire x1="248.92" y1="116.84" x2="248.92" y2="83.82" width="0.1524" layer="91"/>
 <wire x1="248.92" y1="83.82" x2="264.16" y2="83.82" width="0.1524" layer="91"/>
 <junction x="248.92" y="116.84"/>
-</segment>
-</net>
+<pinref part="C6" gate="G$1" pin="P$2"/>
+<wire x1="294.64" y1="83.82" x2="294.64" y2="73.66" width="0.1524" layer="91"/>
+<junction x="294.64" y="73.66"/>
+</segment>
+</net>

Commit message: tweak sent to fab
Parts:
- C1, C6, C7: value .33u -> .47u
- C13, C14: value (none) -> 1u
- R1: value 1M 2kV -> 2M 2kV
- R10: value 3k -> 3k3; device jaw:R1206 -> jaw:R0603
- R23, R24: value (none) -> 4r7
- R3, R4: value 330k -> 392k
- R5: value 3k -> 3k3
Other:
- moved on the sheet: C7
Changed lines of the file:
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@@
 <part name="FRAME1" library="frames" deviceset="FRAME_B_L" device=""/>
 <part name="L1" library="jaw" deviceset="L" device="AIRD03" value="100u"/>
-<part name="C1" library="jaw" deviceset="C" device="R46KI333000N1M" value=".33u"/>
+<part name="C1" library="jaw" deviceset="C" device="R46KI333000N1M" value=".47u"/>
 <part name="C2" library="jaw" deviceset="C" device="MKP1848S62010JY5F" value="20u"/>
 <part name="C3" library="jaw" deviceset="C" device="2220" value=".1u"/>
-<part name="R1" library="jaw" deviceset="R" device="2512" value="1M 2kV"/>
+<part name="R1" library="jaw" deviceset="R" device="2512" value="2M 2kV"/>
 <part name="Q1" library="jaw" deviceset="MOSFET" device="TO247REV" value="MOSFETTO247REV"/>
 <part name="Q3" library="jaw" deviceset="MOSFET" device="TO247REV" value="MOSFETTO247REV"/>
@@
 <part name="L3" library="jaw" deviceset="L" device="2303" value="15u"/>
 <part name="L4" library="jaw" deviceset="L" device="2303" value="15u"/>
-<part name="C6" library="jaw" deviceset="C" device="R46KI333000N1M" value=".33u"/>
-<part name="C7" library="jaw" deviceset="C" device="R46KI333000N1M" value=".33u"/>
-<part name="R5" library="jaw" deviceset="R" device="1206" value="3k"/>
-<part name="R10" library="jaw" deviceset="R" device="1206" value="3k"/>
+<part name="C6" library="jaw" deviceset="C" device="R46KI333000N1M" value=".47u"/>
+<part name="C7" library="jaw" deviceset="C" device="R46KI333000N1M" value=".47u"/>
+<part name="R5" library="jaw" deviceset="R" device="1206" value="3k3"/>
+<part name="R10" library="jaw" deviceset="R" device="0603" value="3k3"/>
 <part name="R12" library="jaw" deviceset="R" device="1206" value="600k"/>
 <part name="CN1" library="jaw" deviceset="HEADER-1X2" device="" value="HEADER-1X2"/>
@@
 <part name="GND12" library="jaw" deviceset="PWR-GND" device=""/>
 <part name="VCCM1" library="jaw" deviceset="PWR-VCCM" device=""/>
-<part name="C13" library="jaw" deviceset="C" device="0603"/>
+<part name="C13" library="jaw" deviceset="C" device="0603" value="1u"/>
 <part name="GND13" library="jaw" deviceset="PWR-GND" device=""/>
-<part name="C14" library="jaw" deviceset="C" device="0603"/>
+<part name="C14" library="jaw" deviceset="C" device="0603" value="1u"/>
 <part name="D3" library="jaw" deviceset="DIODE" device="DO-214AA" value="DIODEDO-214AA"/>
 <part name="VCCM2" library="jaw" deviceset="PWR-VCCM" device=""/>
@@
 <part name="VCC4" library="jaw" deviceset="PWR-VCC" device=""/>
 <part name="VCC5" library="jaw" deviceset="PWR-VCC" device=""/>
-<part name="R3" library="jaw" deviceset="R" device="1206" value="330k"/>
-<part name="R4" library="jaw" deviceset="R" device="1206" value="330k"/>
+<part name="R3" library="jaw" deviceset="R" device="1206" value="392k"/>
+<part name="R4" library="jaw" deviceset="R" device="1206" value="392k"/>
 <part name="R19" library="jaw" deviceset="R" device="0612" value="4r7"/>
 <part name="R20" library="jaw" deviceset="R" device="0612" value="4r7"/>
 <part name="R21" library="jaw" deviceset="R" device="0612" value="4r7"/>
 <part name="R22" library="jaw" deviceset="R" device="0612" value="4r7"/>
-<part name="R23" library="jaw" deviceset="R" device="0612"/>
-<part name="R24" library="jaw" deviceset="R" device="0612"/>
+<part name="R23" library="jaw" deviceset="R" device="0612" value="4r7"/>
+<part name="R24" library="jaw" deviceset="R" device="0612" value="4r7"/>
 <part name="C21" library="jaw" deviceset="C" device="0603" value="1u"/>
 <part name="C22" library="jaw" deviceset="C" device="0603" value="10u"/>
@@
 <instance part="L4" gate="G$1" x="304.8" y="73.66"/>
 <instance part="C6" gate="G$1" x="294.64" y="86.36"/>
-<instance part="C7" gate="G$1" x="312.42" y="86.36"/>
+<instance part="C7" gate="G$1" x="314.96" y="86.36"/>
 <instance part="R5" gate="G$1" x="142.24" y="76.2" rot="R90"/>
 <instance part="R10" gate="G$1" x="335.28" y="86.36" rot="R180"/>
@@
 <instance part="GND6" gate="G$1" x="142.24" y="63.5"/>
 <instance part="GND9" gate="G$1" x="241.3" y="63.5"/>
-<instance part="GND10" gate="G$1" x="320.04" y="83.82"/>
+<instance part="GND10" gate="G$1" x="327.66" y="83.82"/>
 <instance part="C4" gate="G$1" x="121.92" y="86.36"/>
 <instance part="D1" gate="G$1" x="358.14" y="91.44" rot="R270"/>
@@
 <segment>
 <pinref part="GND10" gate="G$1" pin="GND"/>
-<wire x1="320.04" y1="86.36" x2="327.66" y2="86.36" width="0.1524" layer="91"/>
 <pinref part="R10" gate="G$1" pin="P$2"/>
 <wire x1="330.2" y1="86.36" x2="327.66" y2="86.36" width="0.1524" layer="91"/>
@@
 <junction x="358.14" y="99.06"/>
 <pinref part="L3" gate="G$1" pin="P$2"/>
-<wire x1="312.42" y1="99.06" x2="358.14" y2="99.06" width="0.1524" layer="91"/>
+<wire x1="312.42" y1="99.06" x2="314.96" y2="99.06" width="0.1524" layer="91"/>
 <pinref part="C7" gate="G$1" pin="P$1"/>
-<wire x1="312.42" y1="91.44" x2="312.42" y2="99.06" width="0.1524" layer="91"/>
-<junction x="312.42" y="99.06"/>
+<wire x1="314.96" y1="99.06" x2="322.58" y2="99.06" width="0.1524" layer="91"/>
+<wire x1="322.58" y1="99.06" x2="358.14" y2="99.06" width="0.1524" layer="91"/>
+<wire x1="314.96" y1="91.44" x2="314.96" y2="99.06" width="0.1524" layer="91"/>
+<junction x="314.96" y="99.06"/>
 </segment>
 </net>
@@
 <pinref part="C7" gate="G$1" pin="P$2"/>
 <pinref part="L4" gate="G$1" pin="P$2"/>
-<wire x1="312.42" y1="73.66" x2="312.42" y2="83.82" width="0.1524" layer="91"/>
 <pinref part="R3" gate="G$1" pin="P$1"/>
 <wire x1="401.32" y1="76.2" x2="401.32" y2="73.66" width="0.1524" layer="91"/>
 <junction x="401.32" y="73.66"/>
-<wire x1="312.42" y1="73.66" x2="358.14" y2="73.66" width="0.1524" layer="91"/>
-<junction x="312.42" y="73.66"/>
+<wire x1="312.42" y1="73.66" x2="314.96" y2="73.66" width="0.1524" layer="91"/>
+<wire x1="314.96" y1="73.66" x2="358.14" y2="73.66" width="0.1524" layer="91"/>
+<wire x1="314.96" y1="83.82" x2="314.96" y2="73.66" width="0.1524" layer="91"/>
+<junction x="314.96" y="73.66"/>
 </segment>
 </net>

Commit message: tweak text
Parts:
- C19, C20: value (none) -> .1u
- C21: value 1u -> 1u 25V
- C22: value 10u -> 10u 25V
- R5: device jaw:R1206 -> jaw:R0603
Changed lines of the file:
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@@
 <part name="C6" library="jaw" deviceset="C" device="R46KI333000N1M" value=".47u"/>
 <part name="C7" library="jaw" deviceset="C" device="R46KI333000N1M" value=".47u"/>
-<part name="R5" library="jaw" deviceset="R" device="1206" value="3k3"/>
+<part name="R5" library="jaw" deviceset="R" device="0603" value="3k3"/>
 <part name="R10" library="jaw" deviceset="R" device="0603" value="3k3"/>
 <part name="R12" library="jaw" deviceset="R" device="1206" value="600k"/>
@@
 <part name="U9" library="jaw" deviceset="TEMPERATURE" device=""/>
 <part name="U10" library="jaw" deviceset="TEMPERATURE" device=""/>
-<part name="C19" library="jaw" deviceset="C" device="0603"/>
-<part name="C20" library="jaw" deviceset="C" device="0603"/>
+<part name="C19" library="jaw" deviceset="C" device="0603" value=".1u"/>
+<part name="C20" library="jaw" deviceset="C" device="0603" value=".1u"/>
 <part name="GND7" library="jaw" deviceset="PWR-GND" device=""/>
 <part name="GND21" library="jaw" deviceset="PWR-GND" device=""/>
@@
 <part name="R23" library="jaw" deviceset="R" device="0612" value="4r7"/>
 <part name="R24" library="jaw" deviceset="R" device="0612" value="4r7"/>
-<part name="C21" library="jaw" deviceset="C" device="0603" value="1u"/>
-<part name="C22" library="jaw" deviceset="C" device="0603" value="10u"/>
+<part name="C21" library="jaw" deviceset="C" device="0603" value="1u 25V"/>
+<part name="C22" library="jaw" deviceset="C" device="0603" value="10u 25V"/>
 <part name="C23" library="jaw" deviceset="C" device="0603" value="1u"/>
 <part name="C24" library="jaw" deviceset="C" device="0603" value="10u"/>

Commit message: gate snubbers
Parts:
- added D10, D11, D6, D7, D8, D9: DIODESOD-323, jaw:DIODESOD-323
- R19, R20, R21, R22, R23, R24: device jaw:R0612 -> jaw:RSMD0508
Connections:
- net N$19: now also D9.A
- net N$2: now also D9.C
- net N$20: now also D8.A
- net N$21: now also D10.A
- net N$22: now also D11.A
- net N$43: now also D11.C
- net N$44: now also D8.C
- net N$46: now also D10.C
- net N$47: now also D7.C
- net N$48: now also D7.A
- net N$5: now also D6.A
- net N$6: now also D6.C
Other:
- moved on the sheet: C13, C14, C15, C16, C17, C18, D3, D4, D5, R11, R13, R14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
