File: cad/gpi-filter.sch (EAGLE design)
At the start: 13 parts

Commit message: tweak
Parts:
- C3: value .030u -> .027u
- C4: value .010u -> .018u
- C6: value .018u -> .010u
Changed lines of the file:
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@@
 <setting verticaltext="up"/>
 </settings>
-<grid distance="0.1" unitdist="inch" unit="inch" style="lines" multiple="1" display="yes" altdistance="0.01" altunitdist="inch" altunit="inch"/>
+<grid distance="0.1" unitdist="inch" unit="inch" style="lines" multiple="1" display="no" altdistance="0.01" altunitdist="inch" altunit="inch"/>
 <layers>
 <layer number="1" name="Top" color="4" fill="1" visible="no" active="no"/>
@@
 <part name="C1" library="jaw" deviceset="C" device="1210" value=".1"/>
 <part name="C2" library="jaw" deviceset="C" device="1210" value=".1u"/>
-<part name="C3" library="jaw" deviceset="C" device="1210" value=".030u"/>
-<part name="C4" library="jaw" deviceset="C" device="1210" value=".010u"/>
+<part name="C3" library="jaw" deviceset="C" device="1210" value=".027u"/>
+<part name="C4" library="jaw" deviceset="C" device="1210" value=".018u"/>
 <part name="C5" library="jaw" deviceset="C" device="1210" value="DNP"/>
-<part name="C6" library="jaw" deviceset="C" device="1210" value=".018u"/>
+<part name="C6" library="jaw" deviceset="C" device="1210" value=".010u"/>
 <part name="U$1" library="jaw" deviceset="ROBOTMAN-LOGO" device=""/>
 <part name="U$2" library="jaw" deviceset="SYMBOL-WARNING" device=""/>
