File: cad/gpi-top.brd (EAGLE design)
At the start: 130 x 73.5 mm, 2 parts

Commit message: caps
Parts:
- moved U$2 0.25 mm to (26.0, 6.50)
Routing:
- added copper zone on layer 1, net S$1
- added copper zone on layer 16, net S$1
