File: cad/gpi-bottom.brd (EAGLE design)
At the start: 130 x 73.5 mm, 4 parts, among them CN1 HEADER-3X12MM

Commit message: caps
Changed lines of the file:
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@@
 </class>
 </classes>
-<designrules name="default">
+<designrules name="default *">
 <description language="de">&lt;b&gt;EAGLE Design Rules&lt;/b&gt;
 &lt;p&gt;
@@
 <param name="mdViaViaSameLayer" value="8mil"/>
 <param name="mnLayersViaInSmd" value="2"/>
-<param name="mdCopperDimension" value="40mil"/>
+<param name="mdCopperDimension" value="1mil"/>
 <param name="mdDrill" value="8mil"/>
 <param name="mdSmdStop" value="0mil"/>
-<param name="msWidth" value="10mil"/>
+<param name="msWidth" value="0.25mm"/>
 <param name="msDrill" value="24mil"/>
 <param name="msMicroVia" value="9.99mm"/>
@@
 <via x="109.5" y="8.8" extent="1-16" drill="2.5"/>
 <via x="118" y="73" extent="1-16" drill="2"/>
-<via x="127.5" y="15.8" extent="1-16" drill="2.5"/>
 <via x="21.5" y="12.3" extent="1-16" drill="2.5"/>
 <via x="21.5" y="15.8" extent="1-16" drill="2.5"/>

Commit message: comments
Parts:
- moved U$1 38.0 mm to (121.0, 9.00)
Changed lines of the file:
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@@
 <grid distance="0.1" unitdist="mm" unit="mm" style="lines" multiple="10" display="yes" altdistance="0.025" altunitdist="inch" altunit="inch"/>
 <layers>
-<layer number="1" name="Top" color="4" fill="1" visible="yes" active="yes"/>
+<layer number="1" name="Top" color="4" fill="1" visible="no" active="yes"/>
 <layer number="2" name="Route2" color="1" fill="3" visible="no" active="no"/>
 <layer number="3" name="Route3" color="4" fill="3" visible="no" active="no"/>
@@
 <vertex x="-1" y="1"/>
 </polygon>
-<text x="105.5" y="65" size="2" layer="21" ratio="10">JAW 2014-09</text>
-<text x="105.5" y="62" size="1.9" layer="21" ratio="10">www.791rl.com</text>
-<text x="105.5" y="59" size="1.8" layer="21" ratio="10">GPIBOT Rev. 0</text>
-<rectangle x1="105.5" y1="54.1" x2="125.3" y2="58" layer="21"/>
+<text x="108" y="32.1" size="2" layer="21" ratio="10">JAW 2014-09</text>
+<text x="108" y="29" size="1.9" layer="21" ratio="10">www.791rl.com</text>
+<text x="108" y="25.9" size="1.8" layer="21" ratio="10">GPIBOT Rev. 0</text>
+<rectangle x1="108" y1="21" x2="127.8" y2="24.9" layer="21"/>
 </plain>
 <attributes>
@@
 <attribute name="NAME" x="71.8" y="24.2" size="1" layer="25" ratio="10" rot="R90"/>
 </element>
-<element name="U$1" library="jaw" package="ROBOTMAN-LOGO" value="ROBOTMAN-LOGO" x="122" y="47"/>
+<element name="U$1" library="jaw" package="ROBOTMAN-LOGO" value="ROBOTMAN-LOGO" x="121" y="9"/>
 </elements>
 <signals>
 <signal name="S$1">
 <via x="3" y="73" extent="1-16" drill="3.5"/>
-<via x="10" y="73" extent="1-16" drill="2"/>
-<via x="14" y="73" extent="1-16" drill="2"/>
-<via x="22" y="73" extent="1-16" drill="2"/>
-<via x="26" y="73" extent="1-16" drill="2"/>
+<via x="10" y="73" extent="1-16" drill="2.5"/>
+<via x="14" y="73" extent="1-16" drill="2.5"/>
+<via x="22" y="73" extent="1-16" drill="2.5"/>
+<via x="26" y="73" extent="1-16" drill="2.5"/>
 <via x="127" y="73" extent="1-16" drill="3.5"/>
 <via x="3" y="27" extent="1-16" drill="3.5"/>
@@
 <via x="100.5" y="17.55" extent="1-16" drill="2.5"/>
 <via x="100.5" y="7.05" extent="1-16" drill="2.5"/>
-<via x="102" y="73" extent="1-16" drill="2"/>
+<via x="102" y="73" extent="1-16" drill="2.5"/>
 <via x="103.5" y="12.3" extent="1-16" drill="2.5"/>
 <via x="103.5" y="15.8" extent="1-16" drill="2.5"/>
 <via x="103.5" y="8.8" extent="1-16" drill="2.5"/>
-<via x="106" y="73" extent="1-16" drill="2"/>
+<via x="106" y="73" extent="1-16" drill="2.5"/>
 <via x="106.5" y="10.55" extent="1-16" drill="2.5"/>
 <via x="106.5" y="14.05" extent="1-16" drill="2.5"/>
 <via x="106.5" y="17.55" extent="1-16" drill="2.5"/>
 <via x="106.5" y="7.05" extent="1-16" drill="2.5"/>
-<via x="113.9" y="73" extent="1-16" drill="2"/>
+<via x="113.9" y="73" extent="1-16" drill="2.5"/>
 <via x="109.5" y="12.3" extent="1-16" drill="2.5"/>
 <via x="109.5" y="15.8" extent="1-16" drill="2.5"/>
 <via x="109.5" y="8.8" extent="1-16" drill="2.5"/>
-<via x="118" y="73" extent="1-16" drill="2"/>
+<via x="118" y="73" extent="1-16" drill="2.5"/>
 <via x="21.5" y="12.3" extent="1-16" drill="2.5"/>
 <via x="21.5" y="15.8" extent="1-16" drill="2.5"/>
@@
 <via x="30.5" y="17.55" extent="1-16" drill="2.5"/>
 <via x="30.5" y="7.05" extent="1-16" drill="2.5"/>
-<via x="30" y="73" extent="1-16" drill="2"/>
+<via x="30" y="73" extent="1-16" drill="2.5"/>
 <via x="33.5" y="12.3" extent="1-16" drill="2.5"/>
 <via x="33.5" y="15.8" extent="1-16" drill="2.5"/>
 <via x="33.5" y="8.8" extent="1-16" drill="2.5"/>
-<via x="34" y="73" extent="1-16" drill="2"/>
-<via x="38" y="73" extent="1-16" drill="2"/>
+<via x="34" y="73" extent="1-16" drill="2.5"/>
+<via x="38" y="73" extent="1-16" drill="2.5"/>
 <via x="39.5" y="12.3" extent="1-16" drill="2.5"/>
 <via x="39.5" y="15.8" extent="1-16" drill="2.5"/>
@@
 <via x="42.5" y="17.55" extent="1-16" drill="2.5"/>
 <via x="42.5" y="7.05" extent="1-16" drill="2.5"/>
-<via x="42" y="73" extent="1-16" drill="2"/>
+<via x="42" y="73" extent="1-16" drill="2.5"/>
 <via x="45.5" y="12.3" extent="1-16" drill="2.5"/>
 <via x="45.5" y="15.8" extent="1-16" drill="2.5"/>
 <via x="45.5" y="8.8" extent="1-16" drill="2.5"/>
-<via x="46" y="73" extent="1-16" drill="2"/>
+<via x="46" y="73" extent="1-16" drill="2.5"/>
 <via x="48.5" y="10.55" extent="1-16" drill="2.5"/>
 <via x="48.5" y="14.05" extent="1-16" drill="2.5"/>
 <via x="48.5" y="17.55" extent="1-16" drill="2.5"/>
 <via x="48.5" y="7.05" extent="1-16" drill="2.5"/>
-<via x="50" y="73" extent="1-16" drill="2"/>
+<via x="50" y="73" extent="1-16" drill="2.5"/>
 <via x="51.5" y="12.3" extent="1-16" drill="2.5"/>
 <via x="51.5" y="15.8" extent="1-16" drill="2.5"/>
 <via x="51.5" y="8.8" extent="1-16" drill="2.5"/>
-<via x="54" y="73" extent="1-16" drill="2"/>
+<via x="54" y="73" extent="1-16" drill="2.5"/>
 <via x="57.5" y="12.3" extent="1-16" drill="2.5"/>
 <via x="57.5" y="15.8" extent="1-16" drill="2.5"/>
 <via x="57.5" y="8.8" extent="1-16" drill="2.5"/>
-<via x="58" y="73" extent="1-16" drill="2"/>
-<via x="62" y="73" extent="1-16" drill="2"/>
-<via x="60.5" y="14.1" extent="1-16" drill="2.5"/>
-<via x="60.5" y="17.7" extent="1-16" drill="2.5"/>
-<via x="60.5" y="6.9" extent="1-16" drill="2.5"/>
-<via x="60.5" y="10.5" extent="1-16" drill="2.5"/>
+<via x="58" y="73" extent="1-16" drill="2.5"/>
+<via x="62" y="73" extent="1-16" drill="2.5"/>
+<via x="60.5" y="14.05" extent="1-16" drill="2.5"/>
+<via x="60.5" y="17.55" extent="1-16" drill="2.5"/>
+<via x="60.5" y="7.05" extent="1-16" drill="2.5"/>
+<via x="60.5" y="10.55" extent="1-16" drill="2.5"/>
 <via x="66.5" y="10.55" extent="1-16" drill="2.5"/>
 <via x="66.5" y="14.05" extent="1-16" drill="2.5"/>
 <via x="66.5" y="17.55" extent="1-16" drill="2.5"/>
 <via x="66.5" y="7.05" extent="1-16" drill="2.5"/>
-<via x="66" y="73" extent="1-16" drill="2"/>
+<via x="66" y="73" extent="1-16" drill="2.5"/>
 <via x="69.5" y="12.3" extent="1-16" drill="2.5"/>
 <via x="69.5" y="15.8" extent="1-16" drill="2.5"/>
 <via x="69.5" y="8.8" extent="1-16" drill="2.5"/>
-<via x="70" y="73" extent="1-16" drill="2"/>
-<via x="63.5" y="8.85" extent="1-16" drill="2.5"/>
-<via x="63.5" y="12.35" extent="1-16" drill="2.5"/>
-<via x="63.5" y="15.85" extent="1-16" drill="2.5"/>
-<via x="74" y="73" extent="1-16" drill="2"/>
+<via x="70" y="73" extent="1-16" drill="2.5"/>
+<via x="63.5" y="8.8" extent="1-16" drill="2.5"/>
+<via x="63.5" y="12.3" extent="1-16" drill="2.5"/>
+<via x="63.5" y="15.8" extent="1-16" drill="2.5"/>
+<via x="74" y="73" extent="1-16" drill="2.5"/>
 <via x="88.5" y="7.05" extent="1-16" drill="2.5"/>
 <via x="88.5" y="10.55" extent="1-16" drill="2.5"/>
 <via x="88.5" y="14.05" extent="1-16" drill="2.5"/>
-<via x="78" y="73" extent="1-16" drill="2"/>
+<via x="78" y="73" extent="1-16" drill="2.5"/>
 <via x="79.5" y="12.3" extent="1-16" drill="2.5"/>
 <via x="79.5" y="15.8" extent="1-16" drill="2.5"/>
 <via x="79.5" y="8.8" extent="1-16" drill="2.5"/>
-<via x="82" y="73" extent="1-16" drill="2"/>
+<via x="82" y="73" extent="1-16" drill="2.5"/>
 <via x="82.5" y="10.55" extent="1-16" drill="2.5"/>
 <via x="82.5" y="14.05" extent="1-16" drill="2.5"/>
 <via x="82.5" y="17.55" extent="1-16" drill="2.5"/>
 <via x="82.5" y="7.05" extent="1-16" drill="2.5"/>
-<via x="86" y="73" extent="1-16" drill="2"/>
+<via x="86" y="73" extent="1-16" drill="2.5"/>
 <via x="85.5" y="12.3" extent="1-16" drill="2.5"/>
 <via x="85.5" y="15.8" extent="1-16" drill="2.5"/>
 <via x="85.5" y="8.8" extent="1-16" drill="2.5"/>
-<via x="90" y="73" extent="1-16" drill="2"/>
+<via x="90" y="73" extent="1-16" drill="2.5"/>
 <via x="91.5" y="12.3" extent="1-16" drill="2.5"/>
 <via x="91.5" y="15.8" extent="1-16" drill="2.5"/>
 <via x="88.5" y="17.6" extent="1-16" drill="2.5"/>
 <via x="91.5" y="8.8" extent="1-16" drill="2.5"/>
-<via x="94" y="73" extent="1-16" drill="2"/>
-<via x="98" y="73" extent="1-16" drill="2"/>
+<via x="94" y="73" extent="1-16" drill="2.5"/>
+<via x="98" y="73" extent="1-16" drill="2.5"/>
 <via x="97.5" y="12.3" extent="1-16" drill="2.5"/>
 <via x="97.5" y="15.8" extent="1-16" drill="2.5"/>
@@
 <vertex x="-0.9" y="1.9"/>
 </polygon>
+<via x="127" y="5.5" extent="1-16" drill="1.5" diameter="2.5"/>
+<via x="14.1" y="69.7" extent="1-16" drill="2.5"/>
+<via x="18" y="69.7" extent="1-16" drill="2.5"/>
+<via x="114" y="69.8" extent="1-16" drill="2.5"/>
+<via x="110" y="69.8" extent="1-16" drill="2.5"/>
 </signal>
 <signal name="N$1">
@@
 </polygon>
 </signal>
+<signal name="S$2">
+<via x="22" y="69.8" extent="1-16" drill="2.5"/>
+<via x="26" y="69.8" extent="1-16" drill="2.5"/>
+<via x="102" y="69.8" extent="1-16" drill="2.5"/>
+<via x="106" y="69.8" extent="1-16" drill="2.5"/>
+<via x="30" y="69.8" extent="1-16" drill="2.5"/>
+<via x="34" y="69.8" extent="1-16" drill="2.5"/>
+<via x="38" y="69.8" extent="1-16" drill="2.5"/>
+<via x="42" y="69.8" extent="1-16" drill="2.5"/>
+<via x="46" y="69.8" extent="1-16" drill="2.5"/>
+<via x="50" y="69.8" extent="1-16" drill="2.5"/>
+<via x="54" y="69.8" extent="1-16" drill="2.5"/>
+<via x="58" y="69.8" extent="1-16" drill="2.5"/>
+<via x="62" y="69.8" extent="1-16" drill="2.5"/>
+<via x="66" y="69.8" extent="1-16" drill="2.5"/>
+<via x="70" y="69.8" extent="1-16" drill="2.5"/>
+<via x="74" y="69.8" extent="1-16" drill="2.5"/>
+<via x="78" y="69.8" extent="1-16" drill="2.5"/>
+<via x="82" y="69.8" extent="1-16" drill="2.5"/>
+<via x="86" y="69.8" extent="1-16" drill="2.5"/>
+<via x="90" y="69.8" extent="1-16" drill="2.5"/>
+<via x="94" y="69.8" extent="1-16" drill="2.5"/>
+<via x="98" y="69.8" extent="1-16" drill="2.5"/>
+</signal>
 </signals>
