File: cad/gpi-viper.brd (EAGLE design)
At the start: 73.5 x 16 mm, 20 parts, among them CN1 1X4-BIG, CN2 HEADER-1X2.4, U1 VIPER38

Commit message: tweak sent to fab
Routing:
- net N$12: track 52.0 -> 49.6 mm
Other:
- outline, holes or cut-outs redrawn
Changed lines of the file:
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@@
 <board>
 <plain>
-<wire x1="0" y1="0" x2="73.5" y2="0" width="0" layer="20"/>
-<wire x1="73.5" y1="0" x2="73.5" y2="16" width="0" layer="20"/>
-<wire x1="73.5" y1="16" x2="0" y2="16" width="0" layer="20"/>
-<wire x1="0" y1="16" x2="0" y2="0" width="0" layer="20"/>
+<wire x1="0" y1="14" x2="0" y2="2" width="0" layer="20"/>
+<wire x1="0" y1="2" x2="2" y2="0" width="0" layer="20" curve="90"/>
+<wire x1="2" y1="0" x2="71.5" y2="0" width="0" layer="20"/>
+<wire x1="71.5" y1="0" x2="73.5" y2="2" width="0" layer="20" curve="90"/>
+<wire x1="73.5" y1="2" x2="73.5" y2="14" width="0" layer="20"/>
+<wire x1="73.5" y1="14" x2="71.5" y2="16" width="0" layer="20" curve="90"/>
+<wire x1="71.5" y1="16" x2="2" y2="16" width="0" layer="20"/>
+<wire x1="2" y1="16" x2="0" y2="14" width="0" layer="20" curve="90"/>
 <wire x1="12.7" y1="6" x2="12" y2="6" width="0.5" layer="22"/>
 <wire x1="12" y1="6" x2="10" y2="6" width="0.5" layer="22"/>
@@
 <via x="35.3" y="13.8" extent="1-16" drill="0.35"/>
 <via x="36.1" y="8.1" extent="1-16" drill="0.35"/>
-<wire x1="34.4" y1="9" x2="36.1" y2="8.1" width="0" layer="19" extent="1-1"/>
 <via x="39.3" y="12.9" extent="1-16" drill="0.35"/>
 <via x="44.2" y="14.1" extent="1-16" drill="0.35"/>
@@
 <via x="62.5" y="12.8" extent="1-16" drill="0.35"/>
 <via x="68.2" y="8.9" extent="1-16" drill="0.35"/>
-<via x="39.7" y="15.3" extent="1-16" drill="0.35"/>
+<via x="40" y="15.1" extent="1-16" drill="0.35"/>
 <via x="43.2" y="4.1" extent="1-16" drill="0.35"/>
 <via x="46.8" y="3.5" extent="1-16" drill="0.35"/>
@@
 <contactref element="R4" pad="2"/>
 <contactref element="R5" pad="1"/>
-<wire x1="20.5" y1="13.2" x2="22.3" y2="14.9" width="0.5" layer="1"/>
 <contactref element="CN1" pad="1"/>
 <wire x1="23.9" y1="13.1" x2="20.6" y2="13.1" width="0.5" layer="1"/>
@@
 <wire x1="36.6" y1="2.4" x2="24.1" y2="14.9" width="0.5" layer="16"/>
 <via x="24.1" y="14.9" extent="1-16" drill="0.35"/>
-<wire x1="24.1" y1="14.9" x2="22.3" y2="14.9" width="0.5" layer="1"/>
+<wire x1="24.1" y1="14.9" x2="23.9" y2="14.7" width="0.5" layer="1"/>
+<wire x1="23.9" y1="14.7" x2="23.9" y2="13.1" width="0.5" layer="1"/>
 </signal>
 <signal name="N$1">

Commit message: viper package
Parts:
- C4: value 1 -> 1u
- R4: value 590k 500V -> 590k
- moved R4 1.40 mm to (17.7, 13.2)
- moved C2 1.30 mm to (6.04, 2.78)
- moved L1 0.70 mm to (31.5, 5.20)
- moved U$1 0.41 mm to (47.2, 8.70)
- moved U$3 0.30 mm to (8.30, 12.6)
Routing:
- net N$2: track 44.2 -> 42.4 mm
- net N$1: track 9.21 -> 10.8 mm
- net VOUT: track 50.2 -> 48.8 mm
- net N$12: track 49.6 -> 50.9 mm
- net N$7: track 16.0 -> 17.1 mm
- net N$9: track 19.0 -> 18.0 mm
- net N$4: track 28.3 -> 27.4 mm
Other:
- board text added: "GPI1 B2 Rev. 1"
- board text removed: "GPI1 B2 Rev. 0"

Commit message: viper26, clearances, diodes
Parts:
- added C6: .1u 600V, jaw:SMD1210
- added C7: 100u, jaw:SMD1210
- added R1: 3k9, jaw:SMD0603
- C1: value 10u -> .1u
- C3: value .01u -> .1u
- C4: value 1u -> 1
- D1, D2: value DIODEDO-219AB -> 600V ultrafast; device jaw:DO-219AB -> jaw:DO-214AC
- D3: value DIODEDO-219AB -> DIODESOD-323; device jaw:DO-219AB -> jaw:SOD-323
- D4: device jaw:SOD-323 -> jaw:SOD-323@1
- R3, R5: value 3k -> 3k3
- R4: value 590k -> 590k 500V
- U1: value VIPER38 -> VIPER26DIP7; device jaw:VIPER38-P10 -> jaw:VIPER26-P7
- moved R5 26.0 mm to (48.5, 4.00), turned to 0 degrees
- moved U$3 10.6 mm to (2.80, 3.50), flipped to the bottom, turned to 90 degrees
- moved C1 8.64 mm to (23.0, 12.0)
- moved C3 4.04 mm to (32.0, 3.35)
- moved C4 3.60 mm to (47.6, 9.00)
- moved D4 3.50 mm to (49.5, 9.00)
- moved C2 2.52 mm to (8.54, 2.48)
- moved D3 2.47 mm to (28.8, 2.60)
- moved U1 2.25 mm to (14.9, 6.39), turned to 90 degrees
- moved R4 2.10 mm to (15.6, 13.3)
- moved R3 1.68 mm to (25.0, 8.00)
- moved R2 1.53 mm to (25.0, 12.0)
- moved D2 1.46 mm to (30.0, 13.5), turned to 180 degrees
- moved D1 1.44 mm to (30.0, 8.00), turned to 180 degrees
- moved U$1 1.20 mm to (48.0, 9.60)
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Connections:
- new net N$3: C1.2, U1.5
- net GND: now also C6.2, C7.1
- net N$1: now also R1.1; no longer U1.5
- net N$2: now also R1.2; no longer C1.2
- net N$9: now also C6.1; no longer U1.10, U1.6, U1.9
- net VOUT: now also C7.2
Routing:
- net N$1: track 10.8 -> 2.40 mm
- net N$2: track 42.4 -> 34.3 mm
- net GND: track 0.00 -> 6.50 mm, vias 58 -> 47
- net N$4: track 27.4 -> 21.7 mm
- net N$3: track 0.00 -> 5.34 mm
- net VOUT: track 48.8 -> 52.0 mm
- net N$6: track 24.3 -> 26.1 mm
- net N$12: track 50.9 -> 52.4 mm, vias 1 -> 2
- net N$9: track 18.0 -> 19.1 mm
- net N$7: vias 1 -> 2
- added copper zone on layer 16, net N$11
- added copper zone on layer 16, net N$13
- added copper zone on layer 16, net N$14
- added copper zone on layer 16, net N$8
- removed copper zone on layer 1, net N$8
Other:
- outline, holes or cut-outs redrawn

Commit message: tweak
Parts:
- moved R5 0.50 mm to (48.5, 3.50)
Routing:
- net N$12: track 52.4 -> 57.4 mm
- net GND: track 6.50 -> 6.92 mm, vias 47 -> 48
Other:
- board text added: "450V"
- board text added: "Pb"
- board text added: "less unsafe"
- board text added: "very unsafe"
- board text removed: "450V MAX"

Commit message: tweak text
Parts:
- flipped U$1 to the top
Changed lines of the file:
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@@
 <grid distance="0.1" unitdist="mm" unit="mm" style="lines" multiple="10" display="yes" altdistance="0.1" altunitdist="mm" altunit="mm"/>
 <layers>
-<layer number="1" name="Top" color="4" fill="1" visible="yes" active="yes"/>
+<layer number="1" name="Top" color="4" fill="1" visible="no" active="yes"/>
 <layer number="2" name="Route2" color="1" fill="3" visible="no" active="yes"/>
 <layer number="3" name="Route3" color="4" fill="3" visible="no" active="yes"/>
@@
 <attribute name="VALUE" x="46.722" y="1.414" size="1" layer="27" font="vector" ratio="10"/>
 </element>
-<element name="U$1" library="jaw" package="ROBOTMAN-LOGO" value="ROBOTMAN-LOGO" x="48" y="9.6" rot="MR0"/>
+<element name="U$1" library="jaw" package="ROBOTMAN-LOGO" value="ROBOTMAN-LOGO" x="48" y="9.6"/>
 <element name="CN1" library="adafruit" package="1X04-BIG" value="1X4-BIG" x="62.5" y="4" smashed="yes">
 <attribute name="NAME" x="61.1538" y="5.8288" size="1.27" layer="25" ratio="10" display="off"/>

Commit message: labels
Parts:
- flipped U$1 to the bottom
Changed lines of the file:
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@@
 <?xml version="1.0" encoding="utf-8"?>
 <!DOCTYPE eagle SYSTEM "eagle.dtd">
-<eagle version="7.0.1">
+<eagle version="7.1.0">
 <drawing>
 <settings>
@@
 <layer number="23" name="tOrigins" color="15" fill="1" visible="yes" active="yes"/>
 <layer number="24" name="bOrigins" color="15" fill="1" visible="yes" active="yes"/>
-<layer number="25" name="tNames" color="7" fill="1" visible="yes" active="yes"/>
-<layer number="26" name="bNames" color="7" fill="1" visible="yes" active="yes"/>
-<layer number="27" name="tValues" color="7" fill="1" visible="no" active="yes"/>
-<layer number="28" name="bValues" color="7" fill="1" visible="yes" active="yes"/>
+<layer number="25" name="tNames" color="7" fill="1" visible="no" active="yes"/>
+<layer number="26" name="bNames" color="7" fill="1" visible="no" active="yes"/>
+<layer number="27" name="tValues" color="7" fill="1" visible="yes" active="yes"/>
+<layer number="28" name="bValues" color="7" fill="1" visible="no" active="yes"/>
 <layer number="29" name="tStop" color="7" fill="3" visible="no" active="yes"/>
 <layer number="30" name="bStop" color="7" fill="6" visible="no" active="yes"/>
@@
 <elements>
 <element name="U1" library="jaw" package="VIPER26-P7" value="VIPER26DIP7" x="14.93" y="6.39" smashed="yes" rot="R90">
-<attribute name="NAME" x="11.87" y="1.56" size="1" layer="21" ratio="10" rot="R180"/>
+<attribute name="NAME" x="14.67" y="6.76" size="1" layer="21" ratio="10" rot="R180"/>
 </element>
 <element name="D1" library="jaw" package="DO-214AC" value="600V ultrafast" x="30" y="8" smashed="yes" rot="R180">
@@
 <element name="C1" library="jaw" package="SMD0603" value=".1u" x="23" y="12" smashed="yes" rot="R90">
 <attribute name="NAME" x="22.222" y="14.116" size="1" layer="25" font="vector" ratio="10"/>
-<attribute name="VALUE" x="23.468" y="15.176" size="1" layer="27" font="vector" ratio="10" rot="R180"/>
+<attribute name="VALUE" x="22.424" y="13.168" size="1" layer="27" font="vector" ratio="10" rot="R270"/>
 </element>
 <element name="C2" library="jaw" package="SMD0603" value="10u" x="8.54" y="2.48" smashed="yes" rot="R270">
 <attribute name="NAME" x="6.356" y="2.658" size="1" layer="25" font="vector" ratio="10" rot="R270"/>
-<attribute name="VALUE" x="6.454" y="4.258" size="1" layer="27" font="vector" ratio="10" rot="R270"/>
+<attribute name="VALUE" x="8.054" y="3.858" size="1" layer="27" font="vector" ratio="10" rot="R270"/>
 </element>
 <element name="C3" library="jaw" package="SMD0603" value=".1u" x="32.04" y="3.35" smashed="yes" rot="R270">
 <attribute name="NAME" x="31.272" y="0.456" size="1" layer="25" font="vector" ratio="10"/>
-<attribute name="VALUE" x="29.354" y="5.128" size="1" layer="27" font="vector" ratio="10" rot="R270"/>
+<attribute name="VALUE" x="31.554" y="4.628" size="1" layer="27" font="vector" ratio="10" rot="R270"/>
 </element>
 <element name="C4" library="jaw" package="SMD0603" value="1" x="47.6" y="9" smashed="yes" rot="R270">
 <attribute name="NAME" x="46.822" y="6.016" size="1" layer="25" font="vector" ratio="10"/>
-<attribute name="VALUE" x="47.022" y="5.814" size="1" layer="27" font="vector" ratio="10"/>
+<attribute name="VALUE" x="47.422" y="8.114" size="1" layer="27" font="vector" ratio="10"/>
 </element>
 <element name="R1" library="jaw" package="SMD0603" value="3k9" x="23" y="8" smashed="yes" rot="R270">
 <attribute name="NAME" x="21.784" y="6.422" size="1" layer="25" font="vector" ratio="10" rot="R90"/>
-<attribute name="VALUE" x="19.422" y="6.514" size="1" layer="27" font="vector" ratio="10"/>
+<attribute name="VALUE" x="23.486" y="6.822" size="1" layer="27" font="vector" ratio="10" rot="R90"/>
 </element>
 <element name="R2" library="jaw" package="SMD0603" value="10k" x="25" y="12" smashed="yes" rot="R270">
 <attribute name="NAME" x="24.322" y="14.116" size="1" layer="25" font="vector" ratio="10"/>
-<attribute name="VALUE" x="24.362" y="14.274" size="1" layer="27" font="vector" ratio="10"/>
+<attribute name="VALUE" x="25.426" y="10.762" size="1" layer="27" font="vector" ratio="10" rot="R90"/>
 </element>
 <element name="R3" library="jaw" package="SMD0603" value="3k3" x="25" y="8" smashed="yes" rot="R270">
 <attribute name="NAME" x="24.222" y="5.116" size="1" layer="25" font="vector" ratio="10"/>
-<attribute name="VALUE" x="26.572" y="6.384" size="1" layer="27" font="vector" ratio="10"/>
+<attribute name="VALUE" x="25.416" y="6.772" size="1" layer="27" font="vector" ratio="10" rot="R90"/>
 </element>
 <element name="D4" library="jaw" package="SOD-323@1" value="15V" x="49.5" y="9" smashed="yes" rot="R90">
 <attribute name="NAME" x="48.8" y="6" size="1" layer="25" ratio="10"/>
-<attribute name="VALUE" x="50" y="6.484" size="0.4064" layer="27" rot="R180"/>
+<attribute name="VALUE" x="50" y="6.584" size="0.4064" layer="27" rot="R180"/>
 </element>
 <element name="C5" library="jaw" package="SMD1210" value="100u" x="40.5" y="9" smashed="yes" rot="R270">
 <attribute name="NAME" x="39.703" y="11.951" size="1" layer="25" ratio="10"/>
-<attribute name="VALUE" x="38.703" y="4.579" size="1.27" layer="27"/>
+<attribute name="VALUE" x="41.121" y="6.803" size="1.27" layer="27" rot="R90"/>
 </element>
 <element name="CN2" library="jaw" package="HEADER-1X2-THM-WIDE" value="HEADER-1X2.4" x="2.94" y="10.29" smashed="yes" rot="R90">
@@
 <element name="R4" library="jaw" package="SMD1206" value="590k 500V" x="15.6" y="13.3" smashed="yes">
 <attribute name="NAME" x="11.233" y="12.705" size="1" layer="25" ratio="10"/>
-<attribute name="VALUE" x="12.933" y="10.125" size="1.27" layer="27"/>
+<attribute name="VALUE" x="11.133" y="12.625" size="1.27" layer="27"/>
 </element>
 <element name="R5" library="jaw" package="SMD0603" value="3k3" x="48.5" y="3.5" smashed="yes">
 <attribute name="NAME" x="50.522" y="2.916" size="1" layer="25" font="vector" ratio="10"/>
-<attribute name="VALUE" x="46.722" y="1.414" size="1" layer="27" font="vector" ratio="10"/>
-</element>
-<element name="U$1" library="jaw" package="ROBOTMAN-LOGO" value="ROBOTMAN-LOGO" x="48" y="9.6"/>
+<attribute name="VALUE" x="47.322" y="3.114" size="1" layer="27" font="vector" ratio="10"/>
+</element>
+<element name="U$1" library="jaw" package="ROBOTMAN-LOGO" value="ROBOTMAN-LOGO" x="48" y="9.6" rot="MR0"/>
 <element name="CN1" library="adafruit" package="1X04-BIG" value="1X4-BIG" x="62.5" y="4" smashed="yes">
 <attribute name="NAME" x="61.1538" y="5.8288" size="1.27" layer="25" ratio="10" display="off"/>
-<attribute name="VALUE" x="61.23" y="0.825" size="1.27" layer="27"/>
+<attribute name="VALUE" x="61.23" y="0.825" size="1.27" layer="27" display="off"/>
 </element>
 <element name="U$2" library="jaw" package="SYMBOL-WARNING" value="SYMBOL-WARNING" x="2.9" y="3.6" rot="R270"/>
@@
 <element name="C6" library="jaw" package="SMD1210" value=".1u 600V" x="7.6" y="9.5" smashed="yes" rot="R270">
 <attribute name="NAME" x="7.403" y="12.351" size="1" layer="25" ratio="10"/>
-<attribute name="VALUE" x="4.679" y="10.897" size="1.27" layer="27" rot="R270"/>
+<attribute name="VALUE" x="6.979" y="15.797" size="1.27" layer="27" rot="R270"/>
 </element>
 <element name="C7" library="jaw" package="SMD1210" value="100u" x="44.5" y="9" smashed="yes" rot="R270">
 <attribute name="NAME" x="43.803" y="11.951" size="1" layer="25" ratio="10"/>
-<attribute name="VALUE" x="41.579" y="10.397" size="1.27" layer="27" rot="R270"/>
+<attribute name="VALUE" x="43.779" y="11.297" size="1.27" layer="27" rot="R270"/>
 </element>
 </elements>

Commit message: pdfs, comments
Parts:
- C4: value 1 -> 1u
Changed lines of the file:
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@@
 <?xml version="1.0" encoding="utf-8"?>
 <!DOCTYPE eagle SYSTEM "eagle.dtd">
-<eagle version="7.1.0">
+<eagle version="7.2.0">
 <drawing>
 <settings>
@@
 <attribute name="VALUE" x="31.554" y="4.628" size="1" layer="27" font="vector" ratio="10" rot="R270"/>
 </element>
-<element name="C4" library="jaw" package="SMD0603" value="1" x="47.6" y="9" smashed="yes" rot="R270">
+<element name="C4" library="jaw" package="SMD0603" value="1u" x="47.6" y="9" smashed="yes" rot="R270">
 <attribute name="NAME" x="46.822" y="6.016" size="1" layer="25" font="vector" ratio="10"/>
 <attribute name="VALUE" x="47.422" y="8.114" size="1" layer="27" font="vector" ratio="10"/>
