File: cad/gpi-viper.sch (EAGLE design)
At the start: 20 parts, among them CN1 1X4-BIG, CN2 HEADER-1X2.4, U1 VIPER38

Commit message: viper package
Parts:
- C4: value 1 -> 1u
- R4: value 590k 500V -> 590k
Changed lines of the file:
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@@
 <part name="C2" library="jaw" deviceset="C" device="0603" value="10u"/>
 <part name="C3" library="jaw" deviceset="C" device="0603" value=".01u"/>
-<part name="C4" library="jaw" deviceset="C" device="0603" value="1"/>
+<part name="C4" library="jaw" deviceset="C" device="0603" value="1u"/>
 <part name="R2" library="jaw" deviceset="R" device="0603" value="10k"/>
 <part name="R3" library="jaw" deviceset="R" device="0603" value="3k"/>
@@
 <part name="GND3" library="jaw" deviceset="PWR-GND" device=""/>
 <part name="GND4" library="jaw" deviceset="PWR-GND" device=""/>
-<part name="R4" library="jaw" deviceset="R" device="1206" value="590k 500V"/>
+<part name="R4" library="jaw" deviceset="R" device="1206" value="590k"/>
 <part name="R5" library="jaw" deviceset="R" device="0603" value="3k"/>
 <part name="GND6" library="jaw" deviceset="PWR-GND" device=""/>

Commit message: viper26, clearances, diodes
Parts:
- added C6: .1u 600V, jaw:C1210
- added C7: 100u, jaw:C1210
- added R1: 3k9, jaw:R0603
- C1: value 10u -> .1u
- C3: value .01u -> .1u
- C4: value 1u -> 1
- D1, D2: value DIODEDO-219AB -> 600V ultrafast; device jaw:DIODEDO-219AB -> jaw:DIODEDO-214AC
- D3: value DIODEDO-219AB -> DIODESOD-323; device jaw:DIODEDO-219AB -> jaw:DIODESOD-323
- R3, R5: value 3k -> 3k3
- R4: value 590k -> 590k 500V
- U1: value VIPER38 -> VIPER26DIP7; device jaw:VIPER38 -> jaw:VIPER26DIP7
Connections:
- new net N$3: C1.P$2, U1.COMP
- net GND: now also C6.P$2, C7.P$1
- net N$1: now also R1.P$1; no longer U1.EPT
- net N$2: now also R1.P$2; no longer C1.P$2
- net N$9: now also C6.P$1
- net VOUT: now also C7.P$2
Other:
- note added: "Vout = 3.3 * (R2+R3)/R3 + Vdiode"
- moved on the sheet: C1, D4, U1

Commit message: comments
Other:
- note added: "12V out"
Changed lines of the file:
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@@
 <?xml version="1.0" encoding="utf-8"?>
 <!DOCTYPE eagle SYSTEM "eagle.dtd">
-<eagle version="7.0.1">
+<eagle version="7.2.0">
 <drawing>
 <settings>
@@
 <text x="15.24" y="68.58" size="1.778" layer="97">450V DC IN</text>
 <text x="66.04" y="35.56" size="1.778" layer="97">Vout = 3.3 * (R2+R3)/R3 + Vdiode</text>
+<text x="154.94" y="55.88" size="1.778" layer="97">12V out</text>
 </plain>
 <instances>

Commit message: pdfs, comments
Parts:
- C4: value 1 -> 1u
Other:
- note added: "power inverter - 12V board little box challenge"
- note added: "voltage sense - to adc"
Changed lines of the file:
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@@
 <part name="C2" library="jaw" deviceset="C" device="0603" value="10u"/>
 <part name="C3" library="jaw" deviceset="C" device="0603" value=".1u"/>
-<part name="C4" library="jaw" deviceset="C" device="0603" value="1"/>
+<part name="C4" library="jaw" deviceset="C" device="0603" value="1u"/>
 <part name="R1" library="jaw" deviceset="R" device="0603" value="3k9"/>
 <part name="R2" library="jaw" deviceset="R" device="0603" value="10k"/>
@@
 <text x="66.04" y="35.56" size="1.778" layer="97">Vout = 3.3 * (R2+R3)/R3 + Vdiode</text>
 <text x="154.94" y="55.88" size="1.778" layer="97">12V out</text>
+<text x="175.26" y="25.4" size="2.54" layer="94" ratio="10">power inverter - 12V board
+little box challenge</text>
+<text x="86.36" y="91.44" size="1.778" layer="97" ratio="10">voltage sense - to adc</text>
 </plain>
 <instances>
